File: board/hydra-16.kicad_pcb (KiCad board)
At the start: 2 copper layers, 237 x 149.5 mm, 85 parts, among them IC1 74LS189, IC2 74LS189, IC3 74LS189, IC4 SN74LS189AN, J1 Conn_01x32, J2 Conn_01x24, J3 DE9_Plug, U1 74F573, U10 74LS154, U11 74F00, U12 74F02, U13 74F08, U14 74F32, U15 74F30, U16 74LS260, U17 74LS154, U18 7404, U19 628512_DIP32, U2 74F541, U20 628512_DIP32, U21 628512_DIP32, U22 628512_DIP32, U23 74LS139, U24 74F20, U25 74F02, U26 74LS154, U27 74HC138, U28 AT29C040, U29 AT29C040, U3 AT28C64B, U30 AT29C040, U31 AT29C040, U32 AT29C040, U33 AT29C040, U34 AT29C040, U35 AT29C040, U4 W65C02SxP, U5 6522, U6 6551, U7 MAX232, U8 628512_DIP32, U9 74LS154

Commit message: Fixing pin assignments
Parts:
- C1, C2, C3, C4, C5: footprint Capacitor_THT:CP_Radial_Tantal_D4.5mm_P2.50mm -> Capacitor_THT:C_Disc_D5.0mm_W2.5mm_P2.50mm
- IC4: value SN74LS189AN -> 74LS189
- moved C35 59.9 mm to (168.9, 160.0), turned to 0 degrees
- moved U1 55.5 mm to (176.5, 155.6), turned to 180 degrees
- moved C34 35.1 mm to (165.6, 106.2), turned to 0 degrees
- moved C25 25.8 mm to (76.7, 157.6), turned to 90 degrees
- moved C13 25.4 mm to (150.3, 132.3), turned to 180 degrees
- moved C21 22.1 mm to (136.2, 132.4)
- moved U27 22.0 mm to (155.2, 106.1)
- moved U23 19.2 mm to (73.5, 150.0), turned to -90 degrees
- moved C24 4.23 mm to (80.7, 146.2), turned to 180 degrees
- moved C4 0.95 mm to (160.4, 35.0)
- moved C2 0.91 mm to (141.2, 35.0)
- moved C3 0.34 mm to (146.8, 35.0)
- moved C23 0.26 mm to (62.8, 146.1)
- moved U5 0.25 mm to (118.5, 24.2)
- moved C43 0.19 mm to (136.4, 100.3)
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Connections:
- IC1 pad 10: D0 -> D2
- IC1 pad 12: D0 -> D3
- IC1 pad 6: D0 -> D1
- IC2 pad 10: D0 -> D7
- IC2 pad 12: D0 -> D6
- IC2 pad 4: D0 -> D4
- IC2 pad 6: D0 -> D5
- IC3 pad 10: D0 -> D2
- IC3 pad 12: D0 -> D3
- IC3 pad 6: D0 -> D1
- IC4 pad 10: D0 -> D7
- IC4 pad 12: D0 -> D6
- IC4 pad 4: D0 -> D4
- IC4 pad 6: D0 -> D5
- J2 pad 2: D0 -> D1
- J2 pad 3: D0 -> D2
- J2 pad 4: D0 -> D3
- J2 pad 5: D0 -> D4
- J2 pad 6: D0 -> D5
- J2 pad 7: D0 -> D6
- J2 pad 8: D0 -> D7
- U1 pad 3: D0 -> D1
- U1 pad 4: D0 -> D2
- U1 pad 5: D0 -> D3
- U1 pad 6: D0 -> D4
- U1 pad 7: D0 -> D5
- U1 pad 8: D0 -> D6
- U1 pad 9: D0 -> D7
- U19 pad 1: RAMB1 -> nRAMB1
- U19 pad 14: D0 -> D1
- U19 pad 15: D0 -> D2
- U19 pad 17: D0 -> D3
- U19 pad 18: D0 -> D4
- U19 pad 19: D0 -> D5
- U19 pad 20: D0 -> D6
- U19 pad 21: D0 -> D7
- U19 pad 30: RAMB0 -> nRAMB0
- U2 pad 11: D0 -> D7
- U2 pad 12: D0 -> D6
- U2 pad 13: D0 -> D5
- U2 pad 14: D0 -> D4
- U2 pad 15: D0 -> D3
- U2 pad 16: D0 -> D2
- U2 pad 17: D0 -> D1
- U20 pad 1: RAMB1 -> nRAMB1
- U20 pad 14: D0 -> D1
- U20 pad 15: D0 -> D2
- U20 pad 17: D0 -> D3
- U20 pad 18: D0 -> D4
- U20 pad 19: D0 -> D5
- U20 pad 20: D0 -> D6
- U20 pad 21: D0 -> D7
- U20 pad 30: RAMB0 -> nRAMB0
- U21 pad 1: RAMB1 -> nRAMB1
- U21 pad 14: D0 -> D1
- U21 pad 15: D0 -> D2
- U21 pad 17: D0 -> D3
- U21 pad 18: D0 -> D4
- U21 pad 19: D0 -> D5
- U21 pad 20: D0 -> D6
- U21 pad 21: D0 -> D7
- U21 pad 30: RAMB0 -> nRAMB0
- U22 pad 1: RAMB1 -> nRAMB1
- U22 pad 14: D0 -> D1
- U22 pad 15: D0 -> D2
- U22 pad 17: D0 -> D3
- U22 pad 18: D0 -> D4
- U22 pad 19: D0 -> D5
- U22 pad 20: D0 -> D6
- U22 pad 21: D0 -> D7
- U22 pad 30: RAMB0 -> nRAMB0
- U23 pad 1: nBRC0_S -> nBRC15_S
- U23 pad 2: RAMB2 -> nRAMB2
- U23 pad 3: RAMB3 -> nRAMB3
- U28 pad 14: D0 -> D1
- U28 pad 15: D0 -> D2
- U28 pad 17: D0 -> D3
- U28 pad 18: D0 -> D4
- U28 pad 19: D0 -> D5
- U28 pad 20: D0 -> D6
- U28 pad 21: D0 -> D7
- U29 pad 14: D0 -> D1
- U29 pad 15: D0 -> D2
- U29 pad 17: D0 -> D3
- U29 pad 18: D0 -> D4
- U29 pad 19: D0 -> D5
- U29 pad 20: D0 -> D6
- U29 pad 21: D0 -> D7
- U3 pad 12: D0 -> D1
- U3 pad 13: D0 -> D2
- U3 pad 15: D0 -> D3
- U3 pad 16: D0 -> D4
- U3 pad 17: D0 -> D5
- U3 pad 18: D0 -> D6
- U3 pad 19: D0 -> D7
- U30 pad 14: D0 -> D1
- U30 pad 15: D0 -> D2
- U30 pad 17: D0 -> D3
- U30 pad 18: D0 -> D4
- U30 pad 19: D0 -> D5
- U30 pad 20: D0 -> D6
- U30 pad 21: D0 -> D7
- U31 pad 14: D0 -> D1
- U31 pad 15: D0 -> D2
- U31 pad 17: D0 -> D3
- U31 pad 18: D0 -> D4
- U31 pad 19: D0 -> D5
- U31 pad 20: D0 -> D6
- U31 pad 21: D0 -> D7
- U32 pad 14: D0 -> D1
- U32 pad 15: D0 -> D2
- U32 pad 17: D0 -> D3
- U32 pad 18: D0 -> D4
- U32 pad 19: D0 -> D5
- U32 pad 20: D0 -> D6
- U32 pad 21: D0 -> D7
- U33 pad 14: D0 -> D1
- U33 pad 15: D0 -> D2
- U33 pad 17: D0 -> D3
- U33 pad 18: D0 -> D4
- U33 pad 19: D0 -> D5
- U33 pad 20: D0 -> D6
- U33 pad 21: D0 -> D7
- U34 pad 14: D0 -> D1
- U34 pad 15: D0 -> D2
- U34 pad 17: D0 -> D3
- U34 pad 18: D0 -> D4
- U34 pad 19: D0 -> D5
- U34 pad 20: D0 -> D6
- U34 pad 21: D0 -> D7
- U35 pad 14: D0 -> D1
- U35 pad 15: D0 -> D2
- U35 pad 17: D0 -> D3
- U35 pad 18: D0 -> D4
- U35 pad 19: D0 -> D5
- U35 pad 20: D0 -> D6
- U35 pad 21: D0 -> D7
- U4 pad 26: D0 -> D7
- U4 pad 27: D0 -> D6
- U4 pad 28: D0 -> D5
- U4 pad 29: D0 -> D4
- U4 pad 30: D0 -> D3
- U4 pad 31: D0 -> D2
- U4 pad 32: D0 -> D1
- U5 pad 26: D0 -> D7
- U5 pad 27: D0 -> D6
- U5 pad 28: D0 -> D5
- U5 pad 29: D0 -> D4
- U5 pad 30: D0 -> D3
- U5 pad 31: D0 -> D2
- U5 pad 32: D0 -> D1
- U6 pad 19: D0 -> D1
- U6 pad 20: D0 -> D2
- U6 pad 21: D0 -> D3
- U6 pad 22: D0 -> D4
- U6 pad 23: D0 -> D5
- U6 pad 24: D0 -> D6
- U6 pad 25: D0 -> D7
- U8 pad 14: D0 -> D1
- U8 pad 15: D0 -> D2
- U8 pad 17: D0 -> D3
- U8 pad 18: D0 -> D4
- U8 pad 19: D0 -> D5
- U8 pad 20: D0 -> D6
- U8 pad 21: D0 -> D7
Other:
- board size 237 x 149.5 mm -> 237 x 152 mm

Commit message: Added clocks and power connector.
Parts:
- added C44: 33pF, Capacitor_THT:C_Disc_D5.0mm_W2.5mm_P2.50mm, F.Cu at (30.9, 106.3)
- added C45: 33pF, Capacitor_THT:C_Disc_D5.0mm_W2.5mm_P2.50mm, F.Cu at (45.9, 106.3)
- added C46: .1uF, Capacitor_THT:C_Disc_D5.0mm_W2.5mm_P2.50mm, F.Cu at (59.9, 91.8)
- added C47: .1uF, Capacitor_THT:C_Disc_D5.0mm_W2.5mm_P2.50mm, F.Cu at (33.5, 91.9)
- added J4: ATX-20, Connector_Molex:Molex_Mini-Fit_Jr_5566-20A_2x10_P4.20mm_Vertical, F.Cu at (90.4, 91.5)
- added R1: 1M, Resistor_THT:R_Axial_DIN0204_L3.6mm_D1.6mm_P5.08mm_Horizontal, F.Cu at (35.8, 102.3)
- added U36: 74HC14, Package_DIP:DIP-14_W7.62mm_LongPads, F.Cu at (36.7, 99.4)
- added U37: 74LS191, Package_DIP:DIP-16_W7.62mm_LongPads, F.Cu at (63.1, 99.3)
- added Y1: 14.31818MHz, Crystal:Crystal_HC18-U_Vertical, F.Cu at (35.9, 106.3)
- U4, U5: footprint Package_DIP:DIP-40_W15.24mm_LongPads -> Package_DIP:DIP-40_W15.24mm_Socket_LongPads
- moved C10 217.2 mm to (26.7, 226.6)
- moved C17 217.2 mm to (85.1, 226.6)
- moved C30 217.2 mm to (46.4, 226.7)
- moved C9 217.2 mm to (65.7, 226.6)
- moved U28 217.2 mm to (100.3, 223.5)
- moved U29 217.2 mm to (80.9, 223.5)
- moved U30 217.2 mm to (61.5, 223.5)
- moved U31 217.2 mm to (42.1, 223.5)
- moved C22 182.2 mm to (246.2, 226.9)
- moved C23 182.2 mm to (226.1, 226.8)
- moved C24 182.2 mm to (244.0, 226.9)
- moved C25 182.2 mm to (240.0, 238.3)
- moved C26 182.2 mm to (206.1, 226.8)
- moved C27 182.2 mm to (186.4, 226.8)
- moved J1 182.2 mm to (184.1, 242.5)
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Connections:
- U10 pad 19: PHI1O -> Net-(U10-~{E0})
- U17 pad 19: PHI1O -> Net-(U10-~{E0})
- U6 pad 2: unconnected-(U6-CS1-Pad2) -> +5V
- U6 pad 6: unconnected-(U6-XTAL1-Pad6) -> SER_CLK
Other:
- board size 237 x 152 mm -> 247.5 x 163.5 mm

Commit message: More routing changes and board layout optimizations.
Parts:
- added H1: MountingHole, MountingHole:MountingHole_3.2mm_M3, F.Cu at (25.5, 245.5)
- added H10: MountingHole, MountingHole:MountingHole_3.2mm_M3, F.Cu at (182.5, 179.5)
- added H2: MountingHole, MountingHole:MountingHole_3.2mm_M3, F.Cu at (25.5, 90.0)
- added H3: MountingHole, MountingHole:MountingHole_3.2mm_M3, F.Cu at (265.0, 245.5)
- added H4: MountingHole, MountingHole:MountingHole_3.2mm_M3, F.Cu at (139.5, 90.0)
- added H5: MountingHole, MountingHole:MountingHole_3.2mm_M3, F.Cu at (265.0, 90.0)
- added H6: MountingHole, MountingHole:MountingHole_3.2mm_M3, F.Cu at (176.0, 90.0)
- added H7: MountingHole, MountingHole:MountingHole_3.2mm_M3, F.Cu at (141.0, 245.5)
- added H8: MountingHole, MountingHole:MountingHole_3.2mm_M3, F.Cu at (25.5, 158.0)
- added H9: MountingHole, MountingHole:MountingHole_3.2mm_M3, F.Cu at (265.0, 179.5)
- moved IC3 69.9 mm to (141.2, 162.1)
- moved C34 69.9 mm to (162.0, 158.9)
- moved IC1 69.9 mm to (127.2, 162.1)
- moved C43 69.8 mm to (134.8, 158.9)
- moved U27 69.8 mm to (154.4, 162.1)
- moved C36 69.8 mm to (148.8, 158.9)
- moved C33 16.6 mm to (243.7, 120.6)
- moved IC4 16.6 mm to (236.0, 123.8)
- moved C11 14.5 mm to (231.3, 120.6)
- moved U16 14.5 mm to (223.7, 123.8)
- moved C42 12.9 mm to (219.1, 120.6)
- moved U15 12.9 mm to (211.4, 123.8)
- moved C12 6.30 mm to (235.8, 173.9)
- moved U1 6.03 mm to (255.5, 170.5)
- moved U2 6.03 mm to (243.6, 170.6)
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
Commit message: Changing to ATX-sized motherboard with 8 62-pin ISA slots.  Other component connection cleanup as well.
Parts:
- added D1: LED, LED_THT:LED_D3.0mm, F.Cu at (-37.1, 254.0)
- added J10: Bus_Hydra_8bit, PC Edge:TE_7-5530843-0, F.Cu at (-217.3, 88.9)
- added J11: Bus_Hydra_8bit, PC Edge:TE_7-5530843-0, F.Cu at (-237.6, 88.9)
- added J12: Bus_Hydra_8bit, PC Edge:TE_7-5530843-0, F.Cu at (-257.9, 88.9)
- added J13: Bus_Hydra_8bit, PC Edge:TE_7-5530843-0, F.Cu at (-278.2, 88.9)
- added J14: Bus_Hydra_8bit, PC Edge:TE_7-5530843-0, F.Cu at (-298.6, 88.9)
- added J15: Bus_Hydra_8bit, PC Edge:TE_7-5530843-0, F.Cu at (-148.7, 88.9)
- added J16: Bus_Hydra_8bit, PC Edge:TE_7-5530843-0, F.Cu at (-171.6, 88.9)
- added J5: ATX-24, MolexATX24:CON_39299247, F.Cu at (-105.9, 257.4)
- added J6: 0.89488625MHz, Connector_PinHeader_2.54mm:PinHeader_2x01_P2.54mm_Vertical, F.Cu at (-123.6, 75.0)
- added J7: 1.7897725MHz, Connector_PinHeader_2.54mm:PinHeader_2x01_P2.54mm_Vertical, F.Cu at (-118.5, 75.0)
- added J8: 3.579545MHz, Connector_PinHeader_2.54mm:PinHeader_2x01_P2.54mm_Vertical, F.Cu at (-113.5, 75.0)
- added J9: Bus_Hydra_8bit, PC Edge:TE_7-5530843-0, F.Cu at (-194.4, 88.9)
- added R2: 220, Resistor_THT:R_Axial_DIN0204_L3.6mm_D1.6mm_P5.08mm_Horizontal, F.Cu at (-40.8, 259.1)
- added R3: 100, Resistor_THT:R_Axial_DIN0204_L3.6mm_D1.6mm_P5.08mm_Horizontal, F.Cu at (-37.7, 65.5)
- added SW1: PWR_SW, Button_Switch_THT:SW_DIP_SPSTx01_Slide_6.7x4.1mm_W7.62mm_P2.54mm_LowProfile, F.Cu at (-40.6, 263.5)
- added U38: TL074, Package_DIP:DIP-14_W7.62mm_Socket_LongPads, F.Cu at (-32.6, 47.2)
- added U39: YM2151, Package_DIP:DIP-24_W15.24mm_Socket_LongPads, F.Cu at (-69.6, 44.6)
- added U40: YM3012, Package_DIP:DIP-16_W7.62mm_Socket_LongPads, F.Cu at (-45.3, 44.7)
- J4: value ATX-20 -> 7.15909MHz; footprint Connector_Molex:Molex_Mini-Fit_Jr_5566-20A_2x10_P4.20mm_Vertical -> Connector_PinHeader_2.54mm:PinHeader_2x01_P2.54mm_Vertical
- moved H3 591.8 mm to (-288.3, 35.6), turned to 180 degrees
- moved H9 553.5 mm to (-288.3, 165.1), turned to 180 degrees
- moved H5 477.7 mm to (-209.6, 35.6)
- moved C27 457.9 mm to (-273.0, 258.8)
- moved U21 457.9 mm to (-257.8, 255.3)
- moved C26 457.2 mm to (-252.6, 258.8)
- moved U20 457.2 mm to (-237.4, 255.3)
- moved C23 457.0 mm to (-232.4, 258.8)
- moved U19 457.0 mm to (-217.1, 255.3)
- moved C22 456.7 mm to (-212.0, 258.8)
- moved U22 456.7 mm to (-196.8, 255.3)
- moved J1 454.1 mm to (-273.1, 262.9)
- moved J2 454.1 mm to (-262.8, 201.2)
- moved U23 436.7 mm to (-201.9, 205.2)
- moved C25 436.5 mm to (-198.4, 212.8)
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Connections:
- net Net-(U10-~{E0}) renamed nIO_S
- J2 pad 10: +5v -> +5V
- J2 pad 11: +5v -> +5V
- J2 pad 9: +5v -> +5V
- J4 pad 1: +3.3V -> Net-(J4-Pad1)
- J4 pad 2: +3.3V -> PHI2
- U36 pad 10: unconnected-(U36-Pad10) -> Net-(J4-Pad1)
- U36 pad 11: unconnected-(U36-Pad11) -> Net-(U37-Q0)
- U36 pad 12: unconnected-(U36-Pad12) -> HS_CLK
- U36 pad 13: unconnected-(U36-Pad13) -> Net-(U37-Cp)
- U36 pad 4: PHI2 -> SND_CLK
- U36 pad 8: unconnected-(U36-Pad8) -> Net-(J6-Pad1)
- U36 pad 9: unconnected-(U36-Pad9) -> Net-(U37-Q3)
- U37 pad 3: unconnected-(U37-Q0-Pad3) -> Net-(U37-Q0)
- U37 pad 7: unconnected-(U37-Q3-Pad7) -> Net-(U37-Q3)
- U4 pad 1: unconnected-(U4-~{VP}-Pad1) -> VPB
- U4 pad 2: unconnected-(U4-RDY-Pad2) -> RDY
- U4 pad 36: unconnected-(U4-BE-Pad36) -> BE
- U4 pad 5: unconnected-(U4-~{ML}-Pad5) -> MLB
- U4 pad 7: unconnected-(U4-SYNC-Pad7) -> SYNC
- U5 pad 21: IRQB -> IRQ0B
- U6 pad 26: IRQB -> IRQ1B
Other:
- board size 247.5 x 163.5 mm -> 304.8 x 243.8 mm

Commit message: Sample routed PCB with fills.  Not a final version, just an example
Parts:
- H1, H10, H2, H3, H4, H5, H6, H7, H8, H9: footprint MountingHole:MountingHole_3.2mm_M3 -> MountingHole:MountingHole_3.2mm_M3_Pad_TopBottom
- moved C43 26.9 mm to (-294.4, 191.5)
- moved C27 26.9 mm to (-296.0, 244.8)
- moved U21 26.9 mm to (-280.8, 241.3)
- moved U19 26.9 mm to (-240.2, 241.3)
- moved U20 26.9 mm to (-260.5, 241.3)
- moved U22 26.9 mm to (-219.8, 241.3)
- moved C22 26.9 mm to (-235.0, 244.8)
- moved C23 26.9 mm to (-255.4, 244.8)
- moved C26 26.9 mm to (-275.7, 244.8)
- moved IC1 26.9 mm to (-291.0, 199.1)
- moved J2 26.9 mm to (-285.9, 187.2)
- moved J1 26.9 mm to (-296.1, 248.9)
- moved U23 26.9 mm to (-224.9, 191.2)
- moved IC3 26.9 mm to (-265.6, 199.0)
- moved C36 26.9 mm to (-269.3, 191.4)
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Routing:
- net GND: track 0.00 -> 3233.7 mm
- net +5V: track 0.00 -> 2343.6 mm
- net D0: track 0.00 -> 1555.7 mm
- net A3: track 0.00 -> 1451.3 mm
- net RWB: track 0.00 -> 1268.8 mm
- net !RWB: track 0.00 -> 1186.3 mm
- net A10: track 0.00 -> 1162.9 mm
- net A11: track 0.00 -> 1141.3 mm, vias 0 -> 1
- net A6: track 0.00 -> 1134.6 mm
- net A0: track 0.00 -> 1131.7 mm
- net D5: track 0.00 -> 1130.4 mm
- net A5: track 0.00 -> 1060.8 mm, vias 0 -> 1
- net D1: track 0.00 -> 1053.0 mm
- net D2: track 0.00 -> 1041.0 mm
- net A9: track 0.00 -> 1038.2 mm
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- added copper zone on F.Cu, net +5V
- added copper zone on B.Cu, net GND

Commit message: Added surface mount version of memory daughter cards, and lots of schematic updates and fixes, including adding dedicated registers for shared memory bank select at $FFF1 and IRQ vTable entry selector at $FFF2 along with the IRQ vTable registers and priority encoders for 16 IRQs
Parts:
- removed D1: LED, LED_THT:LED_D3.0mm
- removed J16: Bus_Hydra_8bit, PC Edge:TE_7-5530843-0
- removed SW1: PWR_SW, Button_Switch_THT:SW_DIP_SPSTx01_Slide_6.7x4.1mm_W7.62mm_P2.54mm_LowProfile
- added C48: 100uF, Capacitor_THT:CP_Radial_D5.0mm_P2.50mm, F.Cu at (-63.7, 52.1)
- added C49: 100uF, Capacitor_THT:CP_Radial_D5.0mm_P2.50mm, F.Cu at (-46.7, 57.1)
- added C50: .1uF, Capacitor_THT:C_Disc_D5.0mm_W2.5mm_P5.00mm, F.Cu at (-143.5, 64.8)
- added C51: .1uF, Capacitor_THT:C_Disc_D5.0mm_W2.5mm_P5.00mm, F.Cu at (-181.6, 64.8)
- added C52: .1uF, Capacitor_THT:C_Disc_D5.0mm_W2.5mm_P5.00mm, F.Cu at (-156.2, 64.8)
- added C53: .1uF, Capacitor_THT:C_Disc_D5.0mm_W2.5mm_P5.00mm, F.Cu at (-156.2, 91.4)
- added C54: .1uF, Capacitor_THT:C_Disc_D5.0mm_W2.5mm_P5.00mm, F.Cu at (-168.9, 64.8)
- added C55: .1uF, Capacitor_THT:C_Disc_D5.0mm_W2.5mm_P5.00mm, F.Cu at (-143.5, 91.5)
- added C56: .1uF, Capacitor_THT:C_Disc_D5.0mm_W2.5mm_P5.00mm, F.Cu at (-181.6, 91.4)
- added C57: .1uF, Capacitor_THT:C_Disc_D5.0mm_W2.5mm_P5.00mm, F.Cu at (-168.9, 91.5)
- added C58: .1uF, Capacitor_THT:C_Disc_D5.0mm_W2.5mm_P5.00mm, F.Cu at (-138.7, 129.1)
- added C59: .1uF, Capacitor_THT:C_Disc_D5.0mm_W2.5mm_P5.00mm, F.Cu at (-144.8, 159.6)
- added C60: 3300pF, Capacitor_THT:C_Disc_D5.0mm_W2.5mm_P2.50mm, F.Cu at (-57.5, 75.1)
- added C61: 3300pF, Capacitor_THT:C_Disc_D5.0mm_W2.5mm_P2.50mm, F.Cu at (-57.5, 72.0)
- added C62: .1uF, Capacitor_THT:C_Disc_D5.0mm_W2.5mm_P5.00mm, F.Cu at (-50.8, 196.6)
- added C63: .1uF, Capacitor_THT:C_Disc_D5.0mm_W2.5mm_P5.00mm, F.Cu at (-36.8, 196.7)
- added C64: .1uF, Capacitor_THT:C_Disc_D5.0mm_W2.5mm_P5.00mm, F.Cu at (-45.7, 119.4)
- added C65: .1uF, Capacitor_THT:C_Disc_D5.0mm_W2.5mm_P5.00mm, F.Cu at (-31.8, 114.5)
- added C66: .1uF, Capacitor_THT:C_Disc_D5.0mm_W2.5mm_P5.00mm, F.Cu at (-157.5, 159.6)
- added IC5: 74LS189, Package_DIP:DIP-16_W7.62mm_LongPads, F.Cu at (-135.9, 88.9)
- added IC6: 74LS189, Package_DIP:DIP-16_W7.62mm_LongPads, F.Cu at (-148.6, 88.9)
- added IC7: 74LS189, Package_DIP:DIP-16_W7.62mm_LongPads, F.Cu at (-161.3, 88.9)
- added IC8: 74LS189, Package_DIP:DIP-16_W7.62mm_LongPads, F.Cu at (-174.0, 88.9)
- added J17: Front Panel, Connector_PinHeader_2.54mm:PinHeader_2x08_P2.54mm_Vertical, F.Cu at (-299.7, 165.1)
- added RN1: 3.3k, Resistor_THT:R_Array_SIP9, F.Cu at (-171.4, 137.2)
- added U41: DM1813-10, Package_TO_SOT_THT:TO-92L_Inline_Wide, F.Cu at (-293.7, 170.2)
- added U42: 74157, Package_DIP:DIP-16_W7.62mm_LongPads, F.Cu at (-161.3, 61.0)
- added U43: 74157, Package_DIP:DIP-16_W7.62mm_LongPads, F.Cu at (-135.9, 61.0)
- added U44: 74148, Package_DIP:DIP-16_W7.62mm_LongPads, F.Cu at (-174.0, 60.9)
- added U45: 74148, Package_DIP:DIP-16_W7.62mm_LongPads, F.Cu at (-148.6, 60.9)
- added U46: 74F32, Package_DIP:DIP-14_W7.62mm_LongPads, F.Cu at (-131.1, 127.0)
- added U47: 74F573, Package_DIP:DIP-20_W7.62mm_LongPads, F.Cu at (-29.2, 189.1)
- added U48: 74F541, Package_DIP:DIP-20_W7.62mm_LongPads, F.Cu at (-43.2, 189.1)
- added U49: 74F573, Package_DIP:DIP-20_W7.62mm_LongPads, F.Cu at (-24.1, 111.8)
- added U50: 74F541, Package_DIP:DIP-20_W7.62mm_LongPads, F.Cu at (-38.1, 111.8)
- added U51: 74F32, Package_DIP:DIP-14_W7.62mm_LongPads, F.Cu at (-149.9, 157.4)
- added U52: 74F04, Package_DIP:DIP-14_W7.62mm_LongPads, F.Cu at (-137.2, 157.4)
- J15: value Bus_Hydra_8bit -> AudioJack3; footprint PC Edge:TE_7-5530843-0 -> Connector_Audio:Jack_3.5mm_CUI_SJ1-3523N_Horizontal
- R2: value 220 -> 470
- U18: value 7404 -> 74F04
- U23: value 74LS139 -> 74F139
- U27: value 74HC138 -> 74F138
- U36: value 74HC14 -> 74ACT14
- U37: value 74LS191 -> 74F191
- moved R2 264.1 mm to (-293.7, 182.9)
- moved U8 227.1 mm to (-228.6, 187.7), turned to 90 degrees
- moved C6 219.8 mm to (-231.1, 172.5), turned to 180 degrees
- moved C41 208.9 mm to (-261.6, 138.4), turned to 90 degrees
- moved C12 199.9 mm to (-293.4, 137.2)
- moved U10 196.5 mm to (-261.6, 157.5), turned to 90 degrees
- moved U2 189.4 mm to (-290.8, 144.8), turned to 90 degrees
- moved C35 186.0 mm to (-293.4, 149.9), turned to 180 degrees
- moved U1 175.6 mm to (-290.8, 157.5), turned to 90 degrees
- moved C13 145.5 mm to (-171.4, 159.6)
- moved U18 140.9 mm to (-163.8, 157.4), turned to 180 degrees
- moved C8 133.7 mm to (-196.8, 133.4)
- moved C21 123.0 mm to (-130.8, 159.6), turned to -90 degrees
- moved IC2 111.0 mm to (-221.0, 246.4), turned to 180 degrees
- moved J5 108.9 mm to (-11.4, 203.3), turned to -90 degrees
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Connections:
- J1 pad 1: T0 -> unconnected-(J1-Pin_1-Pad1)
- J1 pad 10: B1 -> nRAMB1
- J1 pad 11: B2 -> nRAMB2
- J1 pad 12: B3 -> nRAMB3
- J1 pad 18: nMCS0 -> nBRC0_S
- J1 pad 19: nMCS1 -> nBRC1_S
- J1 pad 2: T1 -> unconnected-(J1-Pin_2-Pad2)
- J1 pad 20: nMCS2 -> nBRC2_S
- J1 pad 21: nMCS3 -> nBRC3_S
- J1 pad 22: nMCS4 -> nBRC4_S
- J1 pad 23: nMCS5 -> nBRC5_S
- J1 pad 24: nMCS6 -> nBRC6_S
- J1 pad 25: nMCS7 -> nBRC7_S
- J1 pad 26: nMCS8 -> nBRC8_S
- J1 pad 27: nMCS9 -> nBRC9_S
- J1 pad 28: nMCS10 -> nBRC10_S
- J1 pad 29: nMCS11 -> nBRC11_S
- J1 pad 3: T2 -> unconnected-(J1-Pin_3-Pad3)
- J1 pad 30: nMCS12 -> nBRC12_S
- J1 pad 31: nMCS13 -> nBRC13_S
- J1 pad 32: nMCS14 -> nBRC14_S
- J1 pad 4: T3 -> unconnected-(J1-Pin_4-Pad4)
- J1 pad 5: T4 -> T0
- J1 pad 6: T5 -> T1
- J1 pad 7: T6 -> T2
- J1 pad 8: T7 -> T3
- J1 pad 9: B0 -> nRAMB0
- J10 pad 13: ~{nIO_S} -> nIO_S
- J10 pad 21: IRQ7B -> SPI_CS3
- J10 pad 22: IRQ6B -> SPI_CS2
- J10 pad 23: IRQ5B -> SPI_CS1
- J10 pad 24: IRQ4B -> SPI_CS0
- J10 pad 25: IRQ3B -> nIOP10_S
- J10 pad 26: SPI_CS3 -> nIOP5_S
- J10 pad 27: SPI_CS2 -> nIRQ10
- J10 pad 28: SPI_CS1 -> nIRQ5
- J10 pad 32: SND_CLK -> nBROMD
- J10 pad 4: IRQ2B -> MLB
- J10 pad 42: ~{nBROF0_S} -> SND_CLK
- J10 pad 43: B3 -> SND_CR
- J10 pad 44: B2 -> SND_CL
- J10 pad 45: B1 -> I2C_SDA
- J10 pad 46: B0 -> I2C_SCL
- J10 pad 6: SPI_CS0 -> BE
- J11 pad 13: ~{nIO_S} -> nIO_S
- J11 pad 21: IRQ7B -> SPI_CS3
- J11 pad 22: IRQ6B -> SPI_CS2
- J11 pad 23: IRQ5B -> SPI_CS1
- J11 pad 24: IRQ4B -> SPI_CS0
- J11 pad 25: IRQ3B -> nIOP11_S
- J11 pad 26: SPI_CS3 -> nIOP6_S
- J11 pad 27: SPI_CS2 -> nIRQ11
- J11 pad 28: SPI_CS1 -> nIRQ6
- J11 pad 32: SND_CLK -> nBROMD
- J11 pad 4: IRQ2B -> MLB
- J11 pad 42: ~{nBROF0_S} -> SND_CLK
- J11 pad 43: B3 -> SND_CR
- J11 pad 44: B2 -> SND_CL
- J11 pad 45: B1 -> I2C_SDA
- J11 pad 46: B0 -> I2C_SCL
- J11 pad 6: SPI_CS0 -> BE
- J12 pad 13: ~{nIO_S} -> nIO_S
- J12 pad 21: IRQ7B -> SPI_CS3
- J12 pad 22: IRQ6B -> SPI_CS2
- J12 pad 23: IRQ5B -> SPI_CS1
- J12 pad 24: IRQ4B -> SPI_CS0
- J12 pad 25: IRQ3B -> nIOP12_S
- J12 pad 26: SPI_CS3 -> nIOP7_S
- J12 pad 27: SPI_CS2 -> nIRQ12
- J12 pad 28: SPI_CS1 -> nIRQ7
- J12 pad 32: SND_CLK -> nBROMD
- J12 pad 4: IRQ2B -> MLB
- J12 pad 42: ~{nBROF0_S} -> SND_CLK
- J12 pad 43: B3 -> SND_CR
- J12 pad 44: B2 -> SND_CL
- J12 pad 45: B1 -> I2C_SDA
- J12 pad 46: B0 -> I2C_SCL
- J12 pad 6: SPI_CS0 -> BE
- J13 pad 13: ~{nIO_S} -> nIO_S
- J13 pad 21: IRQ7B -> SPI_CS3
- J13 pad 22: IRQ6B -> SPI_CS2
- J13 pad 23: IRQ5B -> SPI_CS1
- J13 pad 24: IRQ4B -> SPI_CS0
- J13 pad 25: IRQ3B -> nIOP13_S
- J13 pad 26: SPI_CS3 -> nIOP8_S
- J13 pad 27: SPI_CS2 -> nIRQ13
- J13 pad 28: SPI_CS1 -> nIRQ8
- J13 pad 32: SND_CLK -> nBROMD
- J13 pad 4: IRQ2B -> MLB
- J13 pad 42: ~{nBROF0_S} -> SND_CLK
- J13 pad 43: B3 -> SND_CR
- J13 pad 44: B2 -> SND_CL
- J13 pad 45: B1 -> I2C_SDA
- J13 pad 46: B0 -> I2C_SCL
- J13 pad 6: SPI_CS0 -> BE
- J14 pad 13: ~{nIO_S} -> nIO_S
- J14 pad 21: IRQ7B -> SPI_CS3
- J14 pad 22: IRQ6B -> SPI_CS2
- J14 pad 23: IRQ5B -> SPI_CS1
- J14 pad 24: IRQ4B -> SPI_CS0
- J14 pad 25: IRQ3B -> nIOP14_S
- J14 pad 26: SPI_CS3 -> nIOP9_S
- J14 pad 27: SPI_CS2 -> nIRQ14
- J14 pad 28: SPI_CS1 -> nIRQ9
- J14 pad 32: SND_CLK -> nBROMD
- J14 pad 4: IRQ2B -> MLB
- J14 pad 42: ~{nBROF0_S} -> SND_CLK
- J14 pad 43: B3 -> SND_CR
- J14 pad 44: B2 -> SND_CL
- J14 pad 45: B1 -> I2C_SDA
- J14 pad 46: B0 -> I2C_SCL
- J14 pad 6: SPI_CS0 -> BE
- J9 pad 13: ~{nIO_S} -> nIO_S
- J9 pad 21: IRQ7B -> SPI_CS3
- J9 pad 22: IRQ6B -> SPI_CS2
- J9 pad 23: IRQ5B -> SPI_CS1
- J9 pad 24: IRQ4B -> SPI_CS0
- J9 pad 25: IRQ3B -> nIOP3_S
- J9 pad 26: SPI_CS3 -> nIOP2_S
- J9 pad 27: SPI_CS2 -> nIRQ3
- J9 pad 28: SPI_CS1 -> nIRQ2
- J9 pad 32: SND_CLK -> nBROMD
- J9 pad 4: IRQ2B -> MLB
- J9 pad 42: ~{nBROF0_S} -> SND_CLK
- J9 pad 43: B3 -> SND_CR
- J9 pad 44: B2 -> SND_CL
- J9 pad 45: B1 -> I2C_SDA
- J9 pad 46: B0 -> I2C_SCL
- J9 pad 6: SPI_CS0 -> BE
- R2 pad 1: GND -> Net-(J17-Pin_16)
- R2 pad 2: Net-(D1-K) -> GND
- U10 pad 19: nIO_S -> BROMD
- U14 pad 10: RWB -> A1
- U14 pad 4: A2 -> nFFF0_S
- U14 pad 5: A1 -> RWB
- U14 pad 6: Net-(U13-Pad2) -> Net-(U14-Pad6)
- U14 pad 8: Net-(U14-Pad8) -> Net-(U13-Pad2)
- U14 pad 9: nFFF0_S -> A2
- U17 pad 19: nIO_S -> BROMD
- U18 pad 1: Net-(U14-Pad8) -> Net-(U14-Pad6)
- U18 pad 10: unconnected-(U18-Pad10) -> FFF1_L
- U18 pad 11: unconnected-(U18-Pad11) -> Net-(U18-Pad11)
- U18 pad 8: unconnected-(U18-Pad8) -> BROMD
- U18 pad 9: unconnected-(U18-Pad9) -> nBROMD
- U19 pad 2: T7 -> U3
- U19 pad 28: T4 -> U0
- U19 pad 3: T5 -> U1
- U19 pad 31: T6 -> U2
- U20 pad 2: T7 -> U3
- U20 pad 28: T4 -> U0
- U20 pad 3: T5 -> U1
- U20 pad 31: T6 -> U2
- U21 pad 2: T7 -> U3
- U21 pad 28: T4 -> U0
- U21 pad 3: T5 -> U1
- U21 pad 31: T6 -> U2
- U22 pad 2: T7 -> U3
- U22 pad 28: T4 -> U0
- U22 pad 3: T5 -> U1
- U22 pad 31: T6 -> U2
- U26 pad 1: nBRC0_S -> nBRC15_S
- U26 pad 10: nBRC9_S -> nBRC6_S
- U26 pad 11: nBRC10_S -> nBRC5_S
- U26 pad 13: nBRC11_S -> nBRC4_S
- U26 pad 14: nBRC12_S -> nBRC3_S
- U26 pad 15: nBRC13_S -> nBRC2_S
- U26 pad 16: nBRC14_S -> nBRC1_S
- U26 pad 17: nBRC15_S -> nBRC0_S
- U26 pad 2: nBRC1_S -> nBRC14_S
- U26 pad 3: nBRC2_S -> nBRC13_S
- U26 pad 4: nBRC3_S -> nBRC12_S
- U26 pad 5: nBRC4_S -> nBRC11_S
- U26 pad 6: nBRC5_S -> nBRC10_S
- U26 pad 7: nBRC6_S -> nBRC9_S
- U26 pad 8: nBRC7_S -> nBRC8_S
- U26 pad 9: nBRC8_S -> nBRC7_S
- U27 pad 10: nBROMC5_S -> nBROMC2_S
- U27 pad 11: nBROMC4_S -> nBROMC3_S
- U27 pad 12: nBROMC3_S -> nBROMC4_S
- U27 pad 13: nBROMC2_S -> nBROMC5_S
- U27 pad 14: nBROMC1_S -> nBROMC6_S
- U27 pad 15: nBROMC0_S -> nBROMC7_S
- U27 pad 5: PHI2 -> PHI1O
- U27 pad 7: nBROMC7_S -> nBROMC0_S
- U27 pad 9: nBROMC6_S -> nBROMC1_S
- U38 pad 11: Net-(U38A-VCC-) -> -12V
- U38 pad 13: Net-(U38-Pad13) -> Net-(J15-PadT)
- U38 pad 14: Net-(U38-Pad13) -> Net-(J15-PadT)
- U38 pad 8: Net-(U38-Pad8) -> Net-(J15-PadR)
- U38 pad 9: Net-(U38-Pad8) -> Net-(J15-PadR)
Routing:
- net GND: track 3233.7 -> 0.00 mm
- net +5V: track 2343.6 -> 0.00 mm
- net D0: track 1555.7 -> 0.00 mm
- net A3: track 1451.3 -> 0.00 mm
- net RWB: track 1268.8 -> 0.00 mm
- net !RWB: track 1186.3 -> 0.00 mm
- net A10: track 1162.9 -> 0.00 mm
- net A11: track 1141.3 -> 0.00 mm, vias 1 -> 0
- net A6: track 1134.6 -> 0.00 mm
- net A0: track 1131.7 -> 0.00 mm
- net D5: track 1130.4 -> 0.00 mm
- net A5: track 1060.8 -> 0.00 mm, vias 1 -> 0
- net D1: track 1053.0 -> 0.00 mm
- net D2: track 1041.0 -> 0.00 mm
- net A9: track 1038.2 -> 0.00 mm
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- removed copper zone on F.Cu, net +5V
- removed copper zone on B.Cu, net GND
