File: board/hydra-16.kicad_pcb (KiCad board)
At the start: 2 copper layers, 304.8 x 243.8 mm, 171 parts, among them IC1 74LS189, IC2 74LS189, IC3 74LS189, IC4 74LS189, IC5 74LS219, IC6 74LS219, IC7 74LS219, IC8 74LS219, J1 Conn_01x32, J10 SLOT 1, J11 SLOT 2, J12 SLOT 3, J13 SLOT 4, J14 SLOT 5, J15 AudioJack3, J16 SPI Device 0, J17 Front Panel, J18 SPI Device 1, J19 SPI Device 2, J2 Conn_01x24, J20 SPI Device 3, J21 SPI Device 4, J22 SPI Device 5, J23 SPI Device 6, J24 SPI Device 7, J3 DE9_Plug, J4 7.15909MHz, J5 ATX-24, J6 0.89489MHz, J7 1.78977MHz, J8 3.57955MHz, J9 SLOT 0, U1 74F573, U10 74LS154, U11 74F00, U12 74F86, U13 74F08, U14 74F32, U15 74F30, U16 74LS260, U17 74LS154, U18 74F04, U19 HM628512LP-5, U2 74F541, U20 HM628512LP-5, U21 HM628512LP-5, U22 HM628512LP-5, U23 74F139, U24 74F20, U25 74F02, U26 74LS154, U27 74F138, U28 AT29C040, U29 AT29C040, U3 AT28C64B, U30 AT29C040, U31 AT29C040, U32 AT29C040, U33 AT29C040, U34 AT29C040, U35 AT29C040, U36 74ACT14, U37 74F191, U38 TL074, U39 YM2151, U4 W65C02S, U40 YM3012, U41 DM1813-10, U42 74F157, U43 74F157, U44 74LS148, U45 74LS148, U46 74F32, U47 74F573, U48 74F541, U49 74F573, U5 65C22, U50 74F541, U51 74F32, U52 74F04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

Commit message: Fixing nBROMD routing, removing unnecessary 7404, and minor other cleanup.
Parts:
- removed C59: 104, Capacitor_THT:C_Disc_D5.0mm_W2.5mm_P5.00mm
- removed U52: 74F04, Package_DIP:DIP-14_W7.62mm_Socket_LongPads
- moved R2 24.1 mm to (-6.35, 250.6)
- moved C48 3.14 mm to (-19.2, 202.1), turned to -90 degrees
- moved C67 3.04 mm to (-19.1, 181.5), turned to 90 degrees
- moved U41 0.89 mm to (-15.3, 241.3)
- moved C68 0.42 mm to (-19.1, 166.8)
Connections:
- RN1 pad 8: unconnected-(RN1-R7-Pad8) -> nBROMD
- U10 pad 19: BROMD -> +5V
- U17 pad 19: BROMD -> +5V
- U18 pad 8: BROMD -> FFF2_L
- U18 pad 9: nBROMD -> Net-(U18-Pad9)
- U19 pad 22: Net-(U21-~{CE}) -> Net-(U19-~{CE})
- U21 pad 22: Net-(U19-~{CE}) -> Net-(U21-~{CE})
- U51 pad 11: Net-(U51-Pad11) -> Net-(U18-Pad9)
Routing:
- net +5V: track 0.00 -> 467.5 mm
- net GND: track 0.00 -> 408.5 mm
- net D2: track 0.00 -> 160.2 mm
- net nROMB1: track 0.00 -> 159.1 mm
- net A5: track 0.00 -> 159.1 mm
- net D1: track 0.00 -> 158.9 mm
- net A3: track 0.00 -> 158.9 mm
- net A1: track 0.00 -> 158.9 mm
- net D0: track 0.00 -> 158.7 mm
- net A4: track 0.00 -> 158.6 mm
- net A7: track 0.00 -> 158.5 mm
- net A2: track 0.00 -> 158.4 mm
- net nROMB2: track 0.00 -> 157.9 mm
- net A6: track 0.00 -> 157.9 mm
- net D4: track 0.00 -> 157.9 mm
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
Commit message: Added VIA port A header and voltage protection diode package socket. Updated logic.
Parts:
- added J25: VIA Port A, Connector_PinHeader_2.54mm:PinHeader_2x06_P2.54mm_Vertical, F.Cu at (-27.9, 141.0)
- added J26: SP720APP, Package_DIP:DIP-16_W7.62mm_Socket_LongPads, F.Cu at (-38.1, 141.0)
- J17: footprint Connector_PinHeader_2.54mm:PinHeader_2x08_P2.54mm_Vertical -> Connector_PinHeader_2.54mm:PinHeader_2x06_P2.54mm_Vertical
- U18: value 74F04 -> 74F02
- U25: value 74F02 -> 74LS260
- U38: footprint Package_DIP:DIP-16_W7.62mm_Socket_LongPads -> Package_DIP:CERDIP-14_W7.62mm_SideBrazed_LongPads_Socket
- moved C19 11.5 mm to (-49.5, 95.3)
- moved U5 11.4 mm to (-53.3, 143.5)
- moved U41 3.58 mm to (-17.8, 238.8)
- moved J17 2.40 mm to (-8.77, 228.6)
Connections:
- C18 pad 1: +5V -> Net-(U18E-VCC)
- C65 pad 1: +5V -> GND
- C65 pad 2: GND -> +5V
- J17 pad 10: unconnected-(J17-Pin_10-Pad10) -> GND
- J17 pad 11: RESB -> +5VA
- J17 pad 12: GND -> Net-(J17-Pin_12)
- J17 pad 5: unconnected-(J17-Pin_5-Pad5) -> GND
- J17 pad 6: unconnected-(J17-Pin_6-Pad6) -> GND
- J17 pad 7: unconnected-(J17-Pin_7-Pad7) -> RESB
- J17 pad 8: unconnected-(J17-Pin_8-Pad8) -> +5V
- J17 pad 9: +5V -> Net-(J17-Pin_9)
- J5 pad 16: Net-(J17-Pin_13) -> Net-(J17-Pin_9)
- J5 pad 8: Net-(J17-Pin_15) -> Net-(J5-PWR_OK)
- R2 pad 1: Net-(J17-Pin_16) -> Net-(J17-Pin_12)
- R2 pad 2: GND -> Net-(J5-PWR_OK)
- U11 pad 1: Net-(U11-Pad1) -> unconnected-(U11-Pad1)
- U11 pad 10: nTRA_S -> A15
- U11 pad 2: Net-(U11-Pad2) -> unconnected-(U11-Pad2)
- U11 pad 3: nDPR_S -> unconnected-(U11-Pad3)
- U11 pad 4: nTRA_S -> A15
- U12 pad 10: unconnected-(U12-Pad10) -> A0
- U12 pad 4: unconnected-(U12-Pad4) -> +5V
- U12 pad 5: unconnected-(U12-Pad5) -> RWB
- U12 pad 6: unconnected-(U12-Pad6) -> !RWB
- U12 pad 8: unconnected-(U12-Pad8) -> !A0
- U12 pad 9: unconnected-(U12-Pad9) -> +5V
- U13 pad 11: Net-(U11-Pad13) -> Net-(U13-Pad10)
- U13 pad 12: nTRA_S -> A14
- U13 pad 13: Net-(U13-Pad13) -> A13
- U13 pad 4: A14 -> !RWB
- U13 pad 5: A13 -> nDPR_S0
- U13 pad 6: Net-(U13-Pad13) -> Net-(U13-Pad6)
- U13 pad 8: Net-(U13-Pad8) -> Net-(U11-Pad13)
- U13 pad 9: Net-(U13-Pad9) -> A15
- U14 pad 10: Net-(U13-Pad3) -> Net-(U14-Pad10)
- U14 pad 11: nIO_S -> Net-(U14-Pad10)
- U14 pad 12: Net-(U10-~{E0}) -> nIOP15_S
- U14 pad 13: Net-(U14-Pad13) -> Net-(U13-Pad3)
- U14 pad 4: nFFF0_S -> nIOP15_S
- U14 pad 5: RWB -> nIOB1_S
- U14 pad 6: Net-(U14-Pad6) -> nFFF1_S
- U14 pad 8: Net-(U14-Pad13) -> nIO_S
- U14 pad 9: nIOP15_S -> Net-(U10-~{E0})
- U15 pad 1: nTRA_S -> A15
- U16 pad 1: nTRA_S -> A15
- U16 pad 4: GND -> A6
- U16 pad 5: Net-(U11-Pad1) -> nDPR_S0
- U16 pad 6: Net-(U11-Pad2) -> nDPR_S1
- U18 pad 1: Net-(U14-Pad6) -> FFF0_L
- U18 pad 10: FFF1_L -> FFF2_L
- U18 pad 11: Net-(U18-Pad11) -> A14
- U18 pad 12: !RWB -> A13
- U18 pad 13: RWB -> Net-(U11-Pad5)
- U18 pad 14: +5V -> Net-(U18E-VCC)
- U18 pad 2: FFF0_L -> nFFF0_S
- U18 pad 3: nDPR_S -> RWB
- U18 pad 4: DPR_S -> FFF1_L
- U18 pad 5: A0 -> nFFF1_S
- U18 pad 6: !A0 -> RWB
- U18 pad 8: FFF2_L -> nFFF2_S
- U18 pad 9: Net-(U18-Pad9) -> RWB
- U24 pad 1: DPR_S -> Net-(U13-Pad6)
- U24 pad 10: Net-(U24-Pad10) -> nDPR_S1
- U24 pad 12: Net-(U13-Pad8) -> nDPR_S2
- U24 pad 13: !A0 -> A0
- U24 pad 2: Net-(U24-Pad10) -> nDPR_S1
- U24 pad 4: Net-(U13-Pad8) -> nDPR_S2
- U24 pad 5: A0 -> !A0
- U24 pad 9: DPR_S -> Net-(U13-Pad6)
- U25 pad 1: Net-(U24-Pad10) -> (no net)
- U25 pad 10: Net-(U13-Pad9) -> A3
- U25 pad 11: A14 -> A2
- U25 pad 12: A13 -> (no net)
- U25 pad 13: Net-(U11-Pad5) -> (no net)
- U25 pad 2: A1 -> (no net)
- U25 pad 3: A2 -> (no net)
- U25 pad 4: Net-(U13-Pad10) -> A1
- U25 pad 5: A3 -> (no net)
- U25 pad 6: A4 -> nDPR_S2
- U25 pad 9: A6 -> A4
- U27 pad 6: +5V -> nBROMD
- U46 pad 10: (no net) -> nIOB14_S
- U46 pad 11: Net-(IC5-~{S}) -> nFFF2_S
- U46 pad 13: nIOB14_S -> nIOB2_S
- U46 pad 8: (no net) -> Net-(IC5-~{S})
- U46 pad 9: (no net) -> nIOP15_S
- U5 pad 18: unconnected-(U5-CB1-Pad18) -> CB1
- U5 pad 19: unconnected-(U5-CB2-Pad19) -> CB2
- U5 pad 2: unconnected-(U5-PA0-Pad2) -> PA0
- U5 pad 3: unconnected-(U5-PA1-Pad3) -> PA1
- U5 pad 39: unconnected-(U5-CA2-Pad39) -> CA2
- U5 pad 4: unconnected-(U5-PA2-Pad4) -> PA2
- U5 pad 40: unconnected-(U5-CA1-Pad40) -> CA1
- U5 pad 5: unconnected-(U5-PA3-Pad5) -> PA3
- U5 pad 6: unconnected-(U5-PA4-Pad6) -> PA4
- U5 pad 7: unconnected-(U5-PA5-Pad7) -> PA5
- U5 pad 8: unconnected-(U5-PA6-Pad8) -> PA6
- U5 pad 9: unconnected-(U5-PA7-Pad9) -> PA7
- U8 pad 22: nTRA_S -> A15
- U8 pad 26: unconnected-(U8-A9-Pad26) -> A9
Routing:
- net +5V: track 467.5 -> 0.00 mm
- net GND: track 408.5 -> 0.00 mm
- net D2: track 160.2 -> 0.00 mm
- net nROMB1: track 159.1 -> 0.00 mm
- net A5: track 159.1 -> 0.00 mm
- net D1: track 158.9 -> 0.00 mm
- net A3: track 158.9 -> 0.00 mm
- net A1: track 158.9 -> 0.00 mm
- net D0: track 158.7 -> 0.00 mm
- net A4: track 158.6 -> 0.00 mm
- net A7: track 158.5 -> 0.00 mm
- net A2: track 158.4 -> 0.00 mm
- net nROMB2: track 157.9 -> 0.00 mm
- net A6: track 157.9 -> 0.00 mm
- net D4: track 157.9 -> 0.00 mm
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Other:
- board text added: "CA1 PA7 PA5 PA3 PA1 +5V"
- board text added: "CA2 PA6 PA4 PA2 PA0 GND"
- board text added: "GND +5V"
- board text added: "PLED- PLED+"
- board text added: "PWR- PWR+"
- board text added: "RESET- RESET+"

Commit message: Initial production breakout card and main PCB versions
Parts:
- H11, H12, H13, H14, H15, H16, H17, H18, H19, H20: footprint MountingHole:MountingHole_4mm_Pad_TopBottom -> MountingHole:MountingHole_4mm_Pad_Via
- U8: value Task RAM -> Task RAM ($0000-$7FFF)
- moved C20 183.4 mm to (-24.0, 213.4), turned to 180 degrees
- moved U28 159.3 mm to (-190.5, 217.2), turned to 0 degrees
- moved U35 151.9 mm to (-39.4, 217.2), turned to 0 degrees
- moved C32 141.7 mm to (-45.7, 213.4), turned to 180 degrees
- moved C17 132.2 mm to (-175.3, 213.4), turned to 180 degrees
- moved U29 117.7 mm to (-168.9, 217.2), turned to 0 degrees
- moved U42 112.3 mm to (-241.3, 137.2), turned to -90 degrees
- moved U44 112.3 mm to (-241.3, 149.9), turned to -90 degrees
- moved RN2 112.0 mm to (-240.0, 162.6), turned to 180 degrees
- moved U34 110.5 mm to (-61.0, 217.2), turned to 0 degrees
- moved C51 108.9 mm to (-237.5, 157.5), turned to 90 degrees
- moved C54 107.1 mm to (-237.5, 144.8), turned to 90 degrees
- moved C50 104.7 mm to (-175.3, 161.3)
- moved U43 104.7 mm to (-167.6, 157.5)
- moved C52 104.2 mm to (-188.0, 161.3)
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Connections:
- net Net-(J15-PadR) renamed BD6
- net Net-(J15-PadT) renamed BD5
- C18 pad 1: Net-(U18E-VCC) -> +5V
- U18 pad 14: Net-(U18E-VCC) -> +5V
Routing:
- net GND: track 0.00 -> 2973.9 mm
- net +5V: track 0.00 -> 2108.0 mm
- net D5: track 0.00 -> 1203.1 mm, vias 0 -> 2
- net D6: track 0.00 -> 1197.1 mm
- net D3: track 0.00 -> 1187.5 mm, vias 0 -> 2
- net D0: track 0.00 -> 1184.7 mm, vias 0 -> 4
- net D2: track 0.00 -> 1175.9 mm, vias 0 -> 6
- net D1: track 0.00 -> 1142.2 mm, vias 0 -> 3
- net A3: track 0.00 -> 1118.5 mm, vias 0 -> 2
- net D7: track 0.00 -> 1106.4 mm
- net D4: track 0.00 -> 1096.8 mm
- net A0: track 0.00 -> 1014.6 mm, vias 0 -> 1
- net !RWB: track 0.00 -> 1002.3 mm, vias 0 -> 4
- net A1: track 0.00 -> 1000.0 mm, vias 0 -> 3
- net RWB: track 0.00 -> 954.0 mm, vias 0 -> 1
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- added copper zone on F.Cu, net +5V
- added copper zone on B.Cu, net GND
Other:
- board text added: "Banked ROM ($A000-$DFFF)"
- board text added: "Banked Task RAM ($8000-$9FFF) Banks $00-$EF"
- board text added: "Banks $00-$1F"
- board text added: "Banks $20-$3F"
- board text added: "Banks $40-$5F"
- board text added: "Banks $60-$7F"
- board text added: "Banks $80-$9F"
- board text added: "Banks $A0-$BF"
- board text added: "Banks $C0-$DF"
- board text added: "Banks $E0-$FF"
- board text added: "IRQ Vector RAM ($FFFE/F)"
- board text added: "O/S ROM ($E000-$FEFF) ($FFFC/D)"
- board text added: "Shared RAM ($8000-$9FFF) Banks $F0-$FF"
- board text added: "T Register ($FFF0)"
- board text added: "U Register ($FFF1)"
- board text added: "V Register ($FFF2)"
- board text removed: "Banked ROM"
- board text removed: "IRQ Vector RAM"
- board text removed: "O/S ROM"
- board text removed: "Shared RAM"
- board text removed: "T Register"
- board text removed: "U Register"
- board text removed: "V Register"
