File: board/Mixer.kicad_sch (KiCad schematic)
At the start: 7 parts, among them IC9 LF353P

Commit message: 0.8 Not sure what state it is in
Parts:
- added U12: 74F86, Package_DIP:DIP-14_W7.62mm_Socket_LongPads, symbol 74xx:74LS86
- added U17: 7404, symbol 74xx_IEEE:7404
