File: board/Mixer.kicad_sch (KiCad schematic)
At the start: 9 parts, among them IC9 LF353P, U12 74F86, U17 7404

Commit message: Board V1.1G
Parts:
- removed U12: 74F86, Package_DIP:DIP-14_W7.62mm_Socket_LongPads, symbol 74xx:74LS86
- removed U17: 7404, symbol 74xx_IEEE:7404

Commit message: V1.2B: Final for production.
Connections:
- net GND renamed GNDA
Other:
- moved on the sheet: R6, R7, RN5
