File: board/SharedMem.kicad_sch (KiCad schematic)
At the start: 10 parts, among them U25 HM628512LP-5, U26 74F139, U27 HM628512LP-5, U28 HM628512LP-5, U29 HM628512LP-5

Commit message: 1.7C: Logic corrections and placement tweaks
Connections:
- net RAMB0 renamed RAMB_M0
- net RAMB1 renamed RAMB_M1
- net RAMB2 renamed RAMB_M2
- net RAMB3 renamed RAMB_M3
Changed lines of the file:
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@@
 	(title_block
 		(title "Shared RAM Banks")
-		(date "2025-09-18")
-		(rev "1.7A")
+		(date "2025-10-01")
+		(rev "1.7C")
 		(company "Data Tuning")
 		(comment 1 "Hydra 16")
@@
 	)
 	(junction
-		(at 50.8 107.95)
-		(diameter 0)
-		(color 0 0 0 0)
-	)
-	(junction
 		(at 154.94 102.87)
 		(diameter 0)
@@
 	)
 	(junction
-		(at 20.32 105.41)
+		(at 17.78 105.41)
 		(diameter 0)
 		(color 0 0 0 0)
@@
 	)
 	(bus_entry
-		(at 20.32 120.65)
+		(at 17.78 120.65)
 		(size 2.54 2.54)
 		(stroke
@@
 	)
 	(bus_entry
-		(at 20.32 128.27)
+		(at 17.78 128.27)
 		(size 2.54 2.54)
 		(stroke
@@
 	)
 	(bus_entry
-		(at 20.32 92.71)
+		(at 17.78 92.71)
 		(size 2.54 -2.54)
 		(stroke
@@
 	)
 	(bus_entry
-		(at 20.32 95.25)
+		(at 17.78 95.25)
 		(size 2.54 -2.54)
 		(stroke
@@
 	(wire
 		(pts
-			(xy 22.86 92.71) (xy 38.1 92.71)
+			(xy 20.32 92.71) (xy 38.1 92.71)
 		)
 		(stroke
@@
 	(bus
 		(pts
-			(xy 20.32 120.65) (xy 20.32 128.27)
+			(xy 17.78 120.65) (xy 17.78 128.27)
 		)
 		(stroke
@@
 	(bus
 		(pts
-			(xy 20.32 95.25) (xy 20.32 105.41)
+			(xy 17.78 95.25) (xy 17.78 105.41)
 		)
 		(stroke
@@
 	(wire
 		(pts
-			(xy 50.8 107.95) (xy 115.57 107.95)
-		)
-		(stroke
-			(width 0)
-			(type default)
-		)
-	)
-	(wire
-		(pts
 			(xy 81.28 64.77) (xy 90.17 64.77)
 		)
@@
 	(wire
 		(pts
-			(xy 22.86 90.17) (xy 38.1 90.17)
+			(xy 20.32 90.17) (xy 38.1 90.17)
 		)
 		(stroke
@@
 	(bus
 		(pts
-			(xy 20.32 92.71) (xy 20.32 95.25)
+			(xy 17.78 92.71) (xy 17.78 95.25)
 		)
 		(stroke
@@
 	(bus
 		(pts
-			(xy 20.32 105.41) (xy 66.04 105.41)
+			(xy 17.78 105.41) (xy 66.04 105.41)
 		)
 		(stroke
@@
 	(wire
 		(pts
-			(xy 22.86 123.19) (xy 30.48 123.19)
+			(xy 20.32 123.19) (xy 30.48 123.19)
 		)
 		(stroke
@@
 	(wire
 		(pts
-			(xy 22.86 130.81) (xy 30.48 130.81)
+			(xy 20.32 130.81) (xy 30.48 130.81)
 		)
 		(stroke
@@
 	(bus
 		(pts
-			(xy 20.32 105.41) (xy 20.32 120.65)
+			(xy 17.78 105.41) (xy 17.78 120.65)
 		)
 		(stroke
@@
 		)
 	)
-	(label "RAMB0"
+	(label "RAMB_M0"
 		(at 68.58 90.17 0)
 		(effects
@@
 		)
 	)
-	(label "RAMB2"
+	(label "RAMB_M2"
 		(at 24.13 123.19 0)
 		(effects
@@
 		)
 	)
-	(label "RAMB0"
+	(label "RAMB_M0"
 		(at 172.72 90.17 0)
 		(effects
@@
 		)
 	)
-	(label "RAMB1"
+	(label "RAMB_M1"
 		(at 172.72 92.71 0)
 		(effects
@@
 		)
 	)
-	(label "RAMB1"
-		(at 22.86 92.71 0)
+	(label "RAMB_M1"
+		(at 20.32 92.71 0)
 		(effects
 			(font
@@
 		)
 	)
-	(label "RAMB3"
+	(label "RAMB_M3"
 		(at 24.13 130.81 0)
 		(effects
@@
 		)
 	)
-	(label "RAMB0"
+	(label "RAMB_M0"
 		(at 120.65 90.17 0)
 		(effects
@@
 		)
 	)
-	(label "RAMB1"
+	(label "RAMB_M1"
 		(at 68.58 92.71 0)
 		(effects
@@
 		)
 	)
-	(label "RAMB1"
+	(label "RAMB_M1"
 		(at 120.65 92.71 0)
 		(effects
@@
 		)
 	)
-	(label "RAMB0"
-		(at 22.86 90.17 0)
+	(label "RAMB_M0"
+		(at 20.32 90.17 0)
 		(effects
 			(font
@@
 		)
 	)
-	(global_label "RAMB[0..7]"
+	(global_label "RAMB_M[0..3]"
 		(shape input)
 		(at 241.3 105.41 0)
@@
 		)
 		(property "Intersheetrefs" "${INTERSHEET_REFS}"
-			(at 254.6872 105.41 0)
+			(at 257.1062 105.41 0)
 			(effects
 				(font
