File: board/SharedMem.kicad_sch (KiCad schematic)
At the start: 8 parts, among them IC1 CY62158H-45ZSXI, IC2 CY62158H-45ZSXI, IC3 CY62158H-45ZSXI, IC4 CY62158H-45ZSXI

Commit message: V2.0 rev 2.0D: clock stretching, OS ROM paging and review fixes
Bus timing:
- New GAL C (U88) generates PHI2/PHI1 and the 3.58 MHz sound clock from
  the 14.318 MHz master, replacing the U35 74F191 divider. J36 now selects
  7.16 or 3.58 MHz.
- Banked RAM, banked ROM and slot I/O ($FF20-$FFEF) get one extra PHI2-low
  period plus 0-3 extra PHI2-high periods set in $FFF5 (GAL D). This
  replaces the on-board RDY wait generator; cards can still pull RDY.
- Write strobes are now hold-time safe: PHI1 comes straight from GAL C
  and RWB_M straight from GAL B2.

Review fixes:
- OS ROM chip enable from a single-level decode, output enable from
  GAL B1; -55 part specified. Full 4K OS ROM paging via GAL G.
- Vector RAM writes only during PHI2; $FFF0-$FFFF no longer slowed.
- YM2151 /WR on RWB_M. U62 removed. RB0-RB7 pull-ups (RN5).
- Slot clocks driven through U56 and U34 with 33R series resistors.
- J38 enables in-system flashing of the banked ROMs.
- W65C22S/W65C51N, AS6C4008, DS1813-5 and CY7C192-25 values; R4 1k.
- J7 pin 8 no longer +5V; +5VA renamed +5VSB; serial handshake loop.
- Sheet titles and revisions, slot symbol pin fixes, and project symbol
  and footprint libraries so the project opens on another machine.

Co-Authored-By: Claude Opus 5.5 <noreply@anthropic.com>
Parts:
- IC1, IC2, IC3, IC4: symbol Cypress_Memories:CY62158H-45ZSXI -> Hydra16:CY62158H-45ZSXI
Connections:
- net !RWB_M renamed !RWB
Other:
- title: ZeroPage $00/$01 Mirror Memory and RAM/ROM Bank Logic -> Banked and Shared RAM ($8000-$9FFF)
Changed lines of the file:
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@@
 	(paper "USLetter")
 	(title_block
-		(title "ZeroPage $00/$01 Mirror Memory and RAM/ROM Bank Logic")
-		(date "2026-01-28")
-		(rev "2.0B")
+		(title "Banked and Shared RAM ($8000-$9FFF)")
+		(date "2026-10-06")
+		(rev "2.0D")
 		(company "Data Tuning")
 		(comment 1 "Hydra 16")
@@
 		)
 	)
-	(global_label "!RWB_M"
+	(global_label "!RWB"
 		(shape input)
 		(at 81.28 118.11 90)
@@
 		)
 	)
-	(global_label "!RWB_M"
+	(global_label "!RWB"
 		(shape input)
 		(at 81.28 26.67 90)
@@
 	)
 	(symbol
-		(lib_id "Cypress_Memories:CY62158H-45ZSXI")
+		(lib_id "Hydra16:CY62158H-45ZSXI")
 		(at 107.95 52.07 0)
 		(unit 1)
@@
 	)
 	(symbol
-		(lib_id "Cypress_Memories:CY62158H-45ZSXI")
+		(lib_id "Hydra16:CY62158H-45ZSXI")
 		(at 46.99 52.07 0)
 		(unit 1)
@@
 	)
 	(symbol
-		(lib_id "Cypress_Memories:CY62158H-45ZSXI")
+		(lib_id "Hydra16:CY62158H-45ZSXI")
 		(at 107.95 143.51 0)
 		(unit 1)
@@
 	)
 	(symbol
-		(lib_id "Cypress_Memories:CY62158H-45ZSXI")
+		(lib_id "Hydra16:CY62158H-45ZSXI")
 		(at 46.99 143.51 0)
 		(unit 1)

Commit message: V2.0: speaker headers, A/D bus fix, layout edits
- On-board speakers LS1/LS2 replaced by 2-pin headers J40 (SPEAKER L)
  and J41 (SPEAKER R) for external mini speakers: pin 1 speaker
  (through R30/R31), pin 2 GNDA; J18 still mutes them
- Connectors: a layout move had joined the A[0..15] and D[0..7] buses
  at two crossings (shorting A0-A7 to D0-D7); buses separated again,
  connectivity matches the previous commit
- Layout edits across the sheets (no other connectivity change)
- PCB updated from the schematic

Co-Authored-By: Claude Opus 5.5 <noreply@anthropic.com>
Other:
- title: Banked and Shared RAM ($8000-$9FFF) -> Expansion Slots, SPI Headers and Port A
Changed lines of the file:
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@@
 	(paper "USLetter")
 	(title_block
-		(title "Banked and Shared RAM ($8000-$9FFF)")
+		(title "Expansion Slots, SPI Headers and Port A")
 		(date "2026-10-06")
 		(rev "2.0D")
