File: board/FFF_Registers.kicad_sch (KiCad schematic)
At the start: 20 parts, among them U48 74F573, U49 74F573, U50 74F573, U51 74F541, U52 74F541, U53 74F541, U54 74F32, U55 74F573, U56 74F541, U57 74F02

Commit message: V1.8C production board
Parts:
- renumbered U51 to U49, U55 to U50, U56 to U51, U49 to U52, U52 to U53, U50 to U54, U53 to U55, U54 to U56
Changed lines of the file:
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@@
 		(title "FFFx Registers and Logic")
 		(date "2025-10-01")
-		(rev "1.7C")
+		(rev "1.8A")
 		(company "Data Tuning")
 		(comment 1 "Hydra 16")
@@
 		(dnp no)
 		(fields_autoplaced yes)
-		(property "Reference" "U54"
+		(property "Reference" "U56"
 			(at 195.58 120.65 0)
 			(effects
@@
 			(project ""
 				(path "/ef29fc71-3fec-48b5-8a1a-46bee537a98c/9c3f9893-75ea-4823-afb7-35bb324a2c9f"
-					(reference "U54")
+					(reference "U56")
 					(unit 3)
 				)
@@
 		(dnp no)
 		(fields_autoplaced yes)
-		(property "Reference" "U55"
-			(at 154.5941 34.29 0)
+		(property "Reference" "U50"
+			(at 154.5433 34.29 0)
 			(effects
 				(font
@@
 		)
 		(property "Value" "74F573"
-			(at 154.5941 36.83 0)
+			(at 154.5433 36.83 0)
 			(effects
 				(font
@@
 			(project "hydra-16"
 				(path "/ef29fc71-3fec-48b5-8a1a-46bee537a98c/9c3f9893-75ea-4823-afb7-35bb324a2c9f"
-					(reference "U55")
+					(reference "U50")
 					(unit 1)
 				)
@@
 		(dnp no)
 		(fields_autoplaced yes)
-		(property "Reference" "U54"
+		(property "Reference" "U56"
 			(at 195.58 90.17 0)
 			(effects
@@
 			(project ""
 				(path "/ef29fc71-3fec-48b5-8a1a-46bee537a98c/9c3f9893-75ea-4823-afb7-35bb324a2c9f"
-					(reference "U54")
+					(reference "U56")
 					(unit 1)
 				)
@@
 		(dnp no)
 		(fields_autoplaced yes)
-		(property "Reference" "U51"
-			(at 105.0641 34.29 0)
+		(property "Reference" "U49"
+			(at 105.0133 34.29 0)
 			(effects
 				(font
@@
 		)
 		(property "Value" "74F541"
-			(at 105.0641 36.83 0)
+			(at 105.0133 36.83 0)
 			(effects
 				(font
@@
 			(project "hydra-16"
 				(path "/ef29fc71-3fec-48b5-8a1a-46bee537a98c/9c3f9893-75ea-4823-afb7-35bb324a2c9f"
-					(reference "U51")
+					(reference "U49")
 					(unit 1)
 				)
@@
 		(dnp no)
 		(fields_autoplaced yes)
-		(property "Reference" "U52"
-			(at 108.8741 100.33 0)
+		(property "Reference" "U53"
+			(at 108.8233 100.33 0)
 			(effects
 				(font
@@
 		)
 		(property "Value" "74F541"
-			(at 108.8741 102.87 0)
+			(at 108.8233 102.87 0)
 			(effects
 				(font
@@
 			(project "hydra-16"
 				(path "/ef29fc71-3fec-48b5-8a1a-46bee537a98c/9c3f9893-75ea-4823-afb7-35bb324a2c9f"
-					(reference "U52")
+					(reference "U53")
 					(unit 1)
 				)
@@
 		(dnp no)
 		(fields_autoplaced yes)
-		(property "Reference" "U54"
+		(property "Reference" "U56"
 			(at 154.94 165.0999 0)
 			(effects
@@
 			(project ""
 				(path "/ef29fc71-3fec-48b5-8a1a-46bee537a98c/9c3f9893-75ea-4823-afb7-35bb324a2c9f"
-					(reference "U54")
+					(reference "U56")
 					(unit 5)
 				)
@@
 		(dnp no)
 		(fields_autoplaced yes)
-		(property "Reference" "U49"
-			(at 63.1541 100.33 0)
+		(property "Reference" "U52"
+			(at 63.1033 100.33 0)
 			(effects
 				(font
@@
 		)
 		(property "Value" "74F573"
-			(at 63.1541 102.87 0)
+			(at 63.1033 102.87 0)
 			(effects
 				(font
@@
 			(project "hydra-16"
 				(path "/ef29fc71-3fec-48b5-8a1a-46bee537a98c/9c3f9893-75ea-4823-afb7-35bb324a2c9f"
-					(reference "U49")
+					(reference "U52")
 					(unit 1)
 				)
@@
 		(dnp no)
 		(fields_autoplaced yes)
-		(property "Reference" "U54"
+		(property "Reference" "U56"
 			(at 195.58 105.41 0)
 			(effects
@@
 			(project ""
 				(path "/ef29fc71-3fec-48b5-8a1a-46bee537a98c/9c3f9893-75ea-4823-afb7-35bb324a2c9f"
-					(reference "U54")
+					(reference "U56")
 					(unit 2)
 				)
@@
 		(dnp no)
 		(fields_autoplaced yes)
-		(property "Reference" "U56"
-			(at 204.1241 34.29 0)
+		(property "Reference" "U51"
+			(at 204.0733 34.29 0)
 			(effects
 				(font
@@
 		)
 		(property "Value" "74F541"
-			(at 204.1241 36.83 0)
+			(at 204.0733 36.83 0)
 			(effects
 				(font
@@
 			(project "hydra-16"
 				(path "/ef29fc71-3fec-48b5-8a1a-46bee537a98c/9c3f9893-75ea-4823-afb7-35bb324a2c9f"
-					(reference "U56")
+					(reference "U51")
 					(unit 1)
 				)
@@
 		(dnp no)
 		(fields_autoplaced yes)
-		(property "Reference" "U54"
+		(property "Reference" "U56"
 			(at 195.58 135.89 0)
 			(effects
@@
 			(project ""
 				(path "/ef29fc71-3fec-48b5-8a1a-46bee537a98c/9c3f9893-75ea-4823-afb7-35bb324a2c9f"
-					(reference "U54")
+					(reference "U56")
 					(unit 4)
 				)
@@
 		(dnp no)
 		(fields_autoplaced yes)
-		(property "Reference" "U50"
-			(at 63.1541 152.4 0)
+		(property "Reference" "U54"
+			(at 63.1033 152.4 0)
 			(effects
 				(font
@@
 		)
 		(property "Value" "74F573"
-			(at 63.1541 154.94 0)
+			(at 63.1033 154.94 0)
 			(effects
 				(font
@@
 			(project "hydra-16"
 				(path "/ef29fc71-3fec-48b5-8a1a-46bee537a98c/9c3f9893-75ea-4823-afb7-35bb324a2c9f"
-					(reference "U50")
+					(reference "U54")
 					(unit 1)
 				)
@@
 		(dnp no)
 		(fields_autoplaced yes)
-		(property "Reference" "U53"
-			(at 108.8741 152.4 0)
+		(property "Reference" "U55"
+			(at 108.8233 152.4 0)
 			(effects
 				(font
@@
 		)
 		(property "Value" "74F541"
-			(at 108.8741 154.94 0)
+			(at 108.8233 154.94 0)
 			(effects
 				(font
@@
 			(project "hydra-16"
 				(path "/ef29fc71-3fec-48b5-8a1a-46bee537a98c/9c3f9893-75ea-4823-afb7-35bb324a2c9f"
-					(reference "U53")
+					(reference "U55")
 					(unit 1)
 				)
