File: board/Buffers.kicad_sch (KiCad schematic)
At the start: 8 parts, among them U58 74F541, U59 74F245, U60 74F541, U61 74F125

Commit message: bodge updates
Other:
- moved on the sheet: C78
Changed lines of the file:
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@@
 	)
 	(junction
-		(at 111.76 96.52)
+		(at 46.99 96.52)
 		(diameter 0)
 		(color 0 0 0 0)
@@
 	)
 	(junction
-		(at 111.76 87.63)
-		(diameter 0)
-		(color 0 0 0 0)
-	)
-	(junction
 		(at 85.09 87.63)
 		(diameter 0)
@@
 	)
 	(junction
+		(at 46.99 87.63)
+		(diameter 0)
+		(color 0 0 0 0)
+	)
+	(junction
 		(at 85.09 96.52)
 		(diameter 0)
@@
 	(wire
 		(pts
-			(xy 34.29 96.52) (xy 76.2 96.52)
+			(xy 34.29 96.52) (xy 46.99 96.52)
 		)
 		(stroke
@@
 	(wire
 		(pts
+			(xy 46.99 87.63) (xy 85.09 87.63)
+		)
+		(stroke
+			(width 0)
+			(type default)
+		)
+	)
+	(wire
+		(pts
 			(xy 59.69 107.95) (xy 59.69 114.3)
 		)
@@
 	(wire
 		(pts
+			(xy 46.99 96.52) (xy 76.2 96.52)
+		)
+		(stroke
+			(width 0)
+			(type default)
+		)
+	)
+	(wire
+		(pts
 			(xy 74.93 139.7) (xy 74.93 152.4)
 		)
@@
 	(wire
 		(pts
-			(xy 111.76 92.71) (xy 111.76 96.52)
+			(xy 46.99 92.71) (xy 46.99 96.52)
 		)
 		(stroke
@@
 	(wire
 		(pts
-			(xy 41.91 87.63) (xy 85.09 87.63)
+			(xy 41.91 87.63) (xy 46.99 87.63)
 		)
 		(stroke
@@
 	(wire
 		(pts
-			(xy 69.85 139.7) (xy 69.85 144.78)
+			(xy 76.2 96.52) (xy 85.09 96.52)
 		)
 		(stroke
@@
 		)
 	)
-	(bus
+	(wire
 		(pts
-			(xy 90.17 82.55) (xy 92.71 82.55)
+			(xy 69.85 139.7) (xy 69.85 144.78)
 		)
 		(stroke
@@
 		)
 	)
-	(wire
+	(bus
 		(pts
-			(xy 160.02 128.27) (xy 158.75 128.27)
+			(xy 90.17 82.55) (xy 92.71 82.55)
 		)
 		(stroke
@@
 	(wire
 		(pts
-			(xy 52.07 107.95) (xy 52.07 114.3)
+			(xy 160.02 128.27) (xy 158.75 128.27)
 		)
 		(stroke
@@
 	(wire
 		(pts
-			(xy 85.09 96.52) (xy 76.2 96.52)
+			(xy 52.07 107.95) (xy 52.07 114.3)
 		)
 		(stroke
@@
 		)
 	)
-	(wire
-		(pts
-			(xy 101.6 87.63) (xy 111.76 87.63)
-		)
-		(stroke
-			(width 0)
-			(type default)
-		)
-	)
 	(bus
 		(pts
@@
 	(wire
 		(pts
-			(xy 85.09 96.52) (xy 111.76 96.52)
+			(xy 55.88 73.66) (xy 55.88 80.01)
 		)
 		(stroke
@@
 	(wire
 		(pts
-			(xy 55.88 73.66) (xy 55.88 80.01)
+			(xy 101.6 137.16) (xy 121.92 137.16)
 		)
 		(stroke
@@
 	(wire
 		(pts
-			(xy 101.6 137.16) (xy 121.92 137.16)
+			(xy 110.49 43.18) (xy 110.49 48.26)
 		)
 		(stroke
@@
 	(wire
 		(pts
-			(xy 110.49 43.18) (xy 110.49 48.26)
+			(xy 101.6 87.63) (xy 121.92 87.63)
 		)
 		(stroke
@@
 	(wire
 		(pts
-			(xy 121.92 87.63) (xy 111.76 87.63)
-		)
-		(stroke
-			(width 0)
-			(type default)
-		)
-	)
-	(wire
-		(pts
 			(xy 101.6 101.6) (xy 101.6 106.68)
 		)
@@
 		)
 	)
+	(wire
+		(pts
+			(xy 85.09 96.52) (xy 121.92 96.52)
+		)
+		(stroke
+			(width 0)
+			(type default)
+		)
+	)
 	(bus
 		(pts
@@
 	(wire
 		(pts
-			(xy 111.76 96.52) (xy 121.92 96.52)
-		)
-		(stroke
-			(width 0)
-			(type default)
-		)
-	)
-	(wire
-		(pts
 			(xy 34.29 87.63) (xy 41.91 87.63)
 		)
@@
 	(symbol
 		(lib_id "Device:C_Small")
-		(at 111.76 90.17 0)
+		(at 46.99 90.17 0)
 		(unit 1)
 		(exclude_from_sim no)
@@
 		(fields_autoplaced yes)
 		(property "Reference" "C78"
-			(at 114.3 88.9062 0)
+			(at 49.53 88.9062 0)
 			(effects
 				(font
@@
 		)
 		(property "Value" "104"
-			(at 114.3 91.4462 0)
+			(at 49.53 91.4462 0)
 			(effects
 				(font
@@
 		)
 		(property "Footprint" "Capacitor_THT:C_Disc_D5.0mm_W2.5mm_P5.00mm"
-			(at 111.76 90.17 0)
+			(at 46.99 90.17 0)
 			(effects
 				(font
@@
 		)
 		(property "Datasheet" "~"
-			(at 111.76 90.17 0)
+			(at 46.99 90.17 0)
 			(effects
 				(font
@@
 		)
 		(property "Description" "Unpolarized capacitor, small symbol"
-			(at 111.76 90.17 0)
+			(at 46.99 90.17 0)
 			(effects
 				(font
