File: board/Buffers.kicad_sch (KiCad schematic)
At the start: 8 parts, among them U58 74F541, U59 74F245, U60 74F541, U61 74F125

Commit message: Board version 1.8D complete
Parts:
- added RN4: 103, Resistor_THT:R_Array_SIP9, symbol Device:R_Network08_US
- U59: value 74F245 -> 74ACT245
Connections:
- net +5V: now also RN4.1 (common)
- net D0: now also RN4.2 (R1)
- net D1: now also RN4.3 (R2)
- net D2: now also RN4.4 (R3)
- net D3: now also RN4.5 (R4)
- net D4: now also RN4.6 (R5)
- net D5: now also RN4.7 (R6)
- net D6: now also RN4.8 (R7)
- net D7: now also RN4.9 (R8)
Other:
- note added: "RN4 (1.8D): 10K pull-ups on D0-D7, so a read that nothing answers (an empty slot) gives $FF. U59 is a 74ACT245: CMOS highs into the CPU."
