File: board/Clocks.kicad_sch (KiCad schematic)
At the start: 31 parts, among them J10 Front Panel, J11 ATX-24, J5 0.89489MHz, J6 1.78977MHz, J7 3.57955MHz, J8 7.15909MHz, U39 74ACT14, U40 74F191, U43 DM1813-10, Y1 14.31818MHz

Commit message: V1.8D board enhancements (1.8C software compatible)
Parts:
- U43: Description_1 IC CURRENT SOURCE 3% TO92-3 -> Reset supervisor (DS1813-10): RESB held low at power-up and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
Other:
- note added: "R28 (1.8D): RDY's pull-up, in place of 1.8C's jumper J4 (WAI pulls RDY low)"
- note removed: "R28 (1.8D): RDY never floats (J4 off, or WAI)"
- moved on the sheet: C56
Changed lines of the file:
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@@
 		(comment 1 "Hydra 16")
 	)
-	(text "R28 (1.8D): RDY never floats\n(J4 off, or WAI)"
+	(text "R28 (1.8D): RDY's pull-up, in place of\n1.8C's jumper J4 (WAI pulls RDY low)"
 		(exclude_from_sim no)
 		(at 205.74 163.83 0)
@@
 	)
 	(junction
-		(at 232.41 102.87)
+		(at 218.44 102.87)
 		(diameter 0)
 		(color 0 0 0 0)
@@
 	(wire
 		(pts
-			(xy 167.64 110.49) (xy 232.41 110.49)
+			(xy 167.64 110.49) (xy 218.44 110.49)
 		)
 		(stroke
@@
 	(wire
 		(pts
-			(xy 210.82 102.87) (xy 227.33 102.87)
+			(xy 210.82 102.87) (xy 213.36 102.87)
 		)
 		(stroke
@@
 	(wire
 		(pts
-			(xy 214.63 99.06) (xy 232.41 99.06)
+			(xy 214.63 99.06) (xy 218.44 99.06)
 		)
 		(stroke
@@
 	(wire
 		(pts
-			(xy 232.41 110.49) (xy 232.41 102.87)
+			(xy 218.44 110.49) (xy 218.44 102.87)
 		)
 		(stroke
@@
 	(wire
 		(pts
-			(xy 232.41 99.06) (xy 232.41 102.87)
+			(xy 218.44 99.06) (xy 218.44 102.87)
 		)
 		(stroke
@@
 			)
 		)
-		(property "Description" "RDY pulled up whether J4 is fitted or not (1.8D)"
+		(property "Description" "RDY pulled up (1.8D: in place of 1.8C's jumper J4)"
 			(at 210.82 147.32 0)
 			(effects
@@
 			)
 		)
-		(property "Description" "IC CURRENT SOURCE 3% TO92-3"
+		(property "Description" "Reset supervisor (DS1813-10): RESB held low at power-up and below 4.35 V"
 			(at 233.68 67.31 0)
 			(effects
@@
 			)
 		)
-		(property "Description_1" "IC CURRENT SOURCE 3% TO92-3"
+		(property "Description_1" "Reset supervisor (DS1813-10): RESB held low at power-up and below 4.35 V"
 			(at 238.76 41.91 0)
 			(effects
@@
 	(symbol
 		(lib_id "Device:C_Polarized_Small_US")
-		(at 229.87 102.87 270)
+		(at 215.9 102.87 270)
 		(unit 1)
 		(exclude_from_sim no)
@@
 		(dnp no)
 		(property "Reference" "C56"
-			(at 227.838 107.95 90)
+			(at 213.868 107.95 90)
 			(effects
 				(font
@@
 		)
 		(property "Value" "107"
-			(at 227.838 105.918 90)
+			(at 213.868 105.918 90)
 			(effects
 				(font
@@
 		)
 		(property "Footprint" "Capacitor_THT:CP_Radial_D6.3mm_P2.50mm"
-			(at 229.87 102.87 0)
+			(at 215.9 102.87 0)
 			(effects
 				(font
@@
 		)
 		(property "Datasheet" "~"
-			(at 229.87 102.87 0)
+			(at 215.9 102.87 0)
 			(effects
 				(font
@@
 		)
 		(property "Description" "Polarized capacitor, small US symbol"
-			(at 229.87 102.87 0)
+			(at 215.9 102.87 0)
 			(effects
 				(font
