File: board/Sound.kicad_sch (KiCad schematic)
At the start: 27 parts, among them IC9 LF353P, J29 Audio In 6, J9 SND CT1/2, U38 YM2151, U41 YM3012, U42 TL074

Commit message: bodge updates
Parts:
- added C49: 475, Capacitor_THT:C_Disc_D5.0mm_W2.5mm_P2.50mm, symbol Device:C_Small
Connections:
- net +5V: now also C49.1
- net GNDA: now also C49.2
Changed lines of the file:
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@@
 	)
 	(junction
+		(at 97.79 67.31)
+		(diameter 0)
+		(color 0 0 0 0)
+	)
+	(junction
 		(at 260.35 67.31)
 		(diameter 0)
@@
 	(wire
 		(pts
-			(xy 36.83 67.31) (xy 102.87 67.31)
+			(xy 34.29 69.85) (xy 93.98 69.85)
 		)
 		(stroke
@@
 	(wire
 		(pts
-			(xy 34.29 69.85) (xy 93.98 69.85)
+			(xy 96.52 97.79) (xy 96.52 99.06)
 		)
 		(stroke
@@
 		)
 	)
-	(wire
+	(bus
 		(pts
-			(xy 96.52 97.79) (xy 96.52 99.06)
+			(xy 43.18 97.79) (xy 43.18 100.33)
 		)
 		(stroke
@@
 		)
 	)
-	(bus
+	(wire
 		(pts
-			(xy 43.18 97.79) (xy 43.18 100.33)
+			(xy 101.6 81.28) (xy 97.79 81.28)
 		)
 		(stroke
@@
 	(wire
 		(pts
+			(xy 97.79 72.39) (xy 97.79 81.28)
+		)
+		(stroke
+			(width 0)
+			(type default)
+		)
+	)
+	(wire
+		(pts
+			(xy 36.83 67.31) (xy 97.79 67.31)
+		)
+		(stroke
+			(width 0)
+			(type default)
+		)
+	)
+	(wire
+		(pts
 			(xy 213.36 54.61) (xy 217.17 54.61)
 		)
@@
 	(wire
 		(pts
+			(xy 97.79 67.31) (xy 102.87 67.31)
+		)
+		(stroke
+			(width 0)
+			(type default)
+		)
+	)
+	(wire
+		(pts
 			(xy 52.07 135.89) (xy 100.33 135.89)
 		)
@@
 	)
 	(symbol
+		(lib_id "Device:C_Small")
+		(at 97.79 69.85 0)
+		(unit 1)
+		(exclude_from_sim no)
+		(in_bom yes)
+		(on_board yes)
+		(dnp no)
+		(property "Reference" "C49"
+			(at 100.076 71.882 0)
+			(effects
+				(font
+					(size 1.27 1.27)
+				)
+				(justify left)
+			)
+		)
+		(property "Value" "475"
+			(at 100.076 69.85 0)
+			(effects
+				(font
+					(size 1.27 1.27)
+				)
+				(justify left)
+			)
+		)
+		(property "Footprint" "Capacitor_THT:C_Disc_D5.0mm_W2.5mm_P2.50mm"
+			(at 97.79 69.85 0)
+			(effects
+				(font
+					(size 1.27 1.27)
+				)
+				(hide yes)
+			)
+		)
+		(property "Datasheet" "~"
+			(at 97.79 69.85 0)
+			(effects
+				(font
+					(size 1.27 1.27)
+				)
+				(hide yes)
+			)
+		)
+		(property "Description" "Unpolarized capacitor, small symbol"
+			(at 97.79 69.85 0)
+			(effects
+				(font
+					(size 1.27 1.27)
+				)
+				(hide yes)
+			)
+		)
+		(pin "2"
+		)
+		(pin "1"
+		)
+		(instances
+			(project "hydra-16"
+				(path "/ef29fc71-3fec-48b5-8a1a-46bee537a98c/18057e61-facc-4a14-82c5-5f534ac6d8bb"
+					(reference "C49")
+					(unit 1)
+				)
+			)
+		)
+	)
+	(symbol
 		(lib_id "Yamaha 2151-3012:YM3012")
 		(at 104.14 102.87 0)
@@
 				)
 				(justify left)
-				(hide yes)
 			)
 		)
