File: board/Sound.kicad_sch (KiCad schematic)
At the start: 35 parts, among them IC9 LF353P, J29 Audio In 6, J9 SND CT1/2, U38 YM2151, U41 YM3012, U42 TL074

Commit message: Board V1.8D: the mixer drives headphones cleanly
IC9 is an NJM4556A (the LF353's pinout; the LF353 current-limits into headphones and distorted).
C90/C91 (10 uF) keep the YM3012's 2.5 V of DC out of the summer. Each output gets 33 ohms in series
(R30/R31), 220 uF non-polar to the jack (C92/C93) and a 10K pull-down (R32/R33); the op-amp's side is
AUDIO_x_AMP. The jack has left on the tip and right on the ring (they were swapped). Checked net by net
against the commit before; ERC unchanged. board/CHANGES-1.8D.md updated.

Co-Authored-By: Claude Opus 5.5 <noreply@anthropic.com>
Parts:
- added C90, C91: 106, Capacitor_THT:CP_Radial_D5.0mm_P2.50mm, symbol Device:C_Polarized_Small_US
- added C92, C93: 227 NP, Capacitor_THT:CP_Radial_D8.0mm_P3.50mm, symbol Device:C_Small
- added R30, R31: 330, Resistor_THT:R_Axial_DIN0207_L6.3mm_D2.5mm_P10.16mm_Horizontal, symbol Device:R
- added R32, R33: 103, Resistor_THT:R_Axial_DIN0207_L6.3mm_D2.5mm_P10.16mm_Horizontal, symbol Device:R
- IC9: value LF353P -> NJM4556AD
Connections:
- net AUDIO_L: now also C92.2, R32.1; no longer IC9.1 (1OUT), R20.1
- net AUDIO_R: now also C93.2, R33.1; no longer IC9.7 (2OUT), R21.2
- net GNDA: now also R32.2, R33.2
- net at U42.13, U42.14: now also C90.1; no longer R5.1
- net at U42.8, U42.9: now also C91.1; no longer R4.1
- new net: C93.1, R31.2
- new net: C92.1, R30.2
- new net: C91.2, R4.1
- new net: C90.2, R5.1
- new net AUDIO_L_AMP: IC9.1 (1OUT), R20.1, R30.1
- new net AUDIO_R_AMP: IC9.7 (2OUT), R21.2, R31.1
Other:
- note added: "1.8D: the mixer. IC9 an NJM4556A (the LF353's pinout; it drives headphones: the LF353 needs 2K or more). C90/C91 keep the YM3012's 2.5 V of DC out of the summer. Each output: 33 ohms (stable into a cable), 220 uF non-polar, a 10K pull-down."
