File: board/Sound.kicad_sch (KiCad schematic)
At the start: 43 parts, among them IC9 NJM4556AD, J29 Audio In 6, J9 SND CT1/2, U38 YM2151, U41 YM3012, U42 TL074

Commit message: V1.8D board enhancements (1.8C software compatible)
Parts:
- removed R10, R11, R12, R14, R15, R16, R17, R18, R8, R9: 103, Resistor_THT:R_Axial_DIN0204_L3.6mm_D1.6mm_P5.08mm_Horizontal, symbol Device:R
- J29: value Audio In 6 -> Audio In
- R29, R30, R31, R32, R33: footprint Resistor_THT:R_Axial_DIN0207_L6.3mm_D2.5mm_P10.16mm_Horizontal -> Resistor_THT:R_Axial_DIN0204_L3.6mm_D1.6mm_P5.08mm_Horizontal
Other:
- moved on the sheet: C90, J29, R13, R5, R6, R7
