File: board/Sound.kicad_sch (KiCad schematic)
At the start: 28 parts, among them IC9 LF353P, J29 Audio In 6, J9 SND CT1/2, U38 YM2151, U41 YM3012, U42 TL074

Commit message: Board version 1.8D complete
Parts:
- removed R10, R11, R12, R14, R15, R16, R17, R18, R8, R9: 103, Resistor_THT:R_Axial_DIN0204_L3.6mm_D1.6mm_P5.08mm_Horizontal, symbol Device:R
- added C80, C81, C82, C83, C84, C85: 104, Capacitor_THT:C_Disc_D5.0mm_W2.5mm_P5.00mm, symbol Device:C_Small
- added C90, C91: 106, Capacitor_THT:CP_Radial_D5.0mm_P2.50mm, symbol Device:C_Polarized_Small_US
- added C92, C93: 227 NP, Capacitor_THT:CP_Radial_D8.0mm_P3.50mm, symbol Device:C_Small
- added R29: 0, Resistor_THT:R_Axial_DIN0204_L3.6mm_D1.6mm_P5.08mm_Horizontal, symbol Device:R
- added R30, R31: 330, Resistor_THT:R_Axial_DIN0204_L3.6mm_D1.6mm_P5.08mm_Horizontal, symbol Device:R
- added R32, R33: 103, Resistor_THT:R_Axial_DIN0204_L3.6mm_D1.6mm_P5.08mm_Horizontal, symbol Device:R
- IC9: value LF353P -> NJM4556AD
- J29: value Audio In 6 -> Audio In
Connections:
- net +12V: now also C82.1, C84.1
- net +5V: now also C80.1, C81.1
- net -12V: now also C83.2, C85.2
- net AUDIO_L: now also C92.2, R32.1; no longer IC9.1 (1OUT), R20.1
- net AUDIO_R: now also C93.2, R33.1; no longer IC9.7 (2OUT), R21.2
- net GND: now also C80.2, C81.2, R29.2
- net GNDA: now also C82.2, C83.1, C84.2, C85.1, R29.1, R32.2, R33.2
- net at U42.13, U42.14: now also C90.1; no longer R5.1
- net at U42.8, U42.9: now also C91.1; no longer R4.1
- new net: C93.1, R31.2
- new net: C92.1, R30.2
- new net: C91.2, R4.1
- new net: C90.2, R5.1
- new net AUDIO_L_AMP: IC9.1 (1OUT), R20.1, R30.1
- new net AUDIO_R_AMP: IC9.7 (2OUT), R21.2, R31.1
Other:
- note added: "1.8D: the mixer. IC9 an NJM4556A (the LF353's pinout; it drives headphones: the LF353 needs 2K or more). C90/C91 keep the YM3012's 2.5 V of DC out of the summer. Each output: 33 ohms (stable into a cable), 220 uF non-polar, a 10K pull-down."
- note added: "Decoupling (1.8D): C80 at the YM2151, C81 at the YM3012, C82/C83 at U42's +12 V/-12 V, C84/C85 at IC9's. R29 (0 ohms, or a ferrite bead) joins GNDA to GND here, beside the YM3012: before, they met only inside the supply."
- moved on the sheet: J29, R13, R5, R6, R7
