File: board/Support.kicad_sch (KiCad schematic)
At the start: 46 parts, among them J37 PWR MODE, Q1 2N7000, U75 74HCU04, U78 CD40106B, U79 CD4013B, U80 L79L05, Y1 14.31818MHz, Y2 1.8432MHz

Commit message: V2.0 rev 2.0D: clock stretching, OS ROM paging and review fixes
Bus timing:
- New GAL C (U88) generates PHI2/PHI1 and the 3.58 MHz sound clock from
  the 14.318 MHz master, replacing the U35 74F191 divider. J36 now selects
  7.16 or 3.58 MHz.
- Banked RAM, banked ROM and slot I/O ($FF20-$FFEF) get one extra PHI2-low
  period plus 0-3 extra PHI2-high periods set in $FFF5 (GAL D). This
  replaces the on-board RDY wait generator; cards can still pull RDY.
- Write strobes are now hold-time safe: PHI1 comes straight from GAL C
  and RWB_M straight from GAL B2.

Review fixes:
- OS ROM chip enable from a single-level decode, output enable from
  GAL B1; -55 part specified. Full 4K OS ROM paging via GAL G.
- Vector RAM writes only during PHI2; $FFF0-$FFFF no longer slowed.
- YM2151 /WR on RWB_M. U62 removed. RB0-RB7 pull-ups (RN5).
- Slot clocks driven through U56 and U34 with 33R series resistors.
- J38 enables in-system flashing of the banked ROMs.
- W65C22S/W65C51N, AS6C4008, DS1813-5 and CY7C192-25 values; R4 1k.
- J7 pin 8 no longer +5V; +5VA renamed +5VSB; serial handshake loop.
- Sheet titles and revisions, slot symbol pin fixes, and project symbol
  and footprint libraries so the project opens on another machine.

Co-Authored-By: Claude Opus 5.5 <noreply@anthropic.com>
Connections:
- net +5VA renamed +5VSB
- net SER_CLK renamed SER_CLK_SRC
Other:
- note added: "DMA: DMAB or BE low releases the bus. GAL B2 (U83) synchronises the request to the end of PHI2, so the CPU clock gate and buffer enables only change while PHI2 is low. Cards drive the bus after that edge."
- note added: "SERIAL CLOCK: Y2 1.8432 MHz Pierce oscillator (U75) -> SER_CLK_SRC -> U34 buffer -> SER_CLK (ACIA); R24 33R -> slot pin 15 (SER_CLK_BUS). BUS CLOCK: Y1 14.31818 MHz on U75 -> U34 squares it -> HS_CLK_SRC -> U88 bus clock generator; R9 33R -> slot HS_CLK."
- note removed: "DMA: DMAB or BE low releases the bus. U77 synchronises the request to the PHI2 falling edge, so the CPU clock gate and buffer enables only change while PHI2 is low. Cards drive the bus after that edge."
- note removed: "SERIAL CLOCK: Y2 1.8432 MHz Pierce oscillator (U75) -> SER_CLK, exact 6551 baud rates; also slot pin 15. BUS CLOCK: Y1 14.31818 MHz on U75 (unbuffered inverter); U34 (Clocks) squares it -> U35 + R9 33R series feed to slots."
- title: Support: Oscillators, DMA Sync, Soft Power, Audio Output, -5V -> Support: Oscillators, Soft Power, Audio Output, -5V
Changed lines of the file:
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@@
 	(paper "A3")
 	(title_block
-		(title "Support: Oscillators, DMA Sync, Soft Power, Audio Output, -5V")
-		(date "2026-10-04")
-		(rev "2.0C")
+		(title "Support: Oscillators, Soft Power, Audio Output, -5V")
+		(date "2026-10-06")
+		(rev "2.0D")
 		(company "Data Tuning")
 		(comment 1 "Hydra 16")
 	)
-	(text "DMA: DMAB or BE low releases the bus. U77 synchronises the request to the PHI2 falling edge,\nso the CPU clock gate and buffer enables only change while PHI2 is low. Cards drive the bus after that edge."
+	(text "DMA: DMAB or BE low releases the bus. GAL B2 (U83) synchronises the request to the end of PHI2,\nso the CPU clock gate and buffer enables only change while PHI2 is low. Cards drive the bus after that edge."
 		(exclude_from_sim no)
 		(at 279.146 127.734 0)
@@
 		)
 	)
-	(text "SERIAL CLOCK: Y2 1.8432 MHz Pierce oscillator (U75) -> SER_CLK, exact 6551 baud rates; also slot pin 15.\nBUS CLOCK: Y1 14.31818 MHz on U75 (unbuffered inverter); U34 (Clocks) squares it -> U35 + R9 33R series feed to slots."
+	(text "SERIAL CLOCK: Y2 1.8432 MHz Pierce oscillator (U75) -> SER_CLK_SRC -> U34 buffer -> SER_CLK (ACIA);\n  R24 33R -> slot pin 15 (SER_CLK_BUS).\nBUS CLOCK: Y1 14.31818 MHz on U75 -> U34 squares it -> HS_CLK_SRC -> U88 bus clock generator;\n  R9 33R -> slot HS_CLK."
 		(exclude_from_sim no)
 		(at 279.146 112.734 0)
@@
 		)
 	)
-	(global_label "SER_CLK"
+	(global_label "SER_CLK_SRC"
 		(shape output)
 		(at 55.88 88.9 0)
@@
 	)
 	(symbol
-		(lib_id "power:+5VA")
+		(lib_id "Hydra16:+5VSB")
 		(at 215.9 171.45 0)
 		(unit 1)
@@
 			)
 		)
-		(property "Value" "+5VA"
+		(property "Value" "+5VSB"
 			(at 215.9 167.64 0)
 			(effects
@@
 	)
 	(symbol
-		(lib_id "power:+5VA")
+		(lib_id "Hydra16:+5VSB")
 		(at 190.5 171.45 0)
 		(unit 1)
@@
 			)
 		)
-		(property "Value" "+5VA"
+		(property "Value" "+5VSB"
 			(at 190.5 167.64 0)
 			(effects
@@
 	)
 	(symbol
-		(lib_id "power:+5VA")
+		(lib_id "Hydra16:+5VSB")
 		(at 279.4 171.45 0)
 		(unit 1)
@@
 			)
 		)
-		(property "Value" "+5VA"
+		(property "Value" "+5VSB"
 			(at 279.4 167.64 0)
 			(effects
@@
 	)
 	(symbol
-		(lib_id "power:+5VA")
+		(lib_id "Hydra16:+5VSB")
 		(at 63.5 119.38 0)
 		(unit 1)
@@
 			)
 		)
-		(property "Value" "+5VA"
+		(property "Value" "+5VSB"
 			(at 63.5 115.57 0)
 			(effects
@@
 	)
 	(symbol
-		(lib_id "power:+5VA")
+		(lib_id "Hydra16:+5VSB")
 		(at 266.7 171.45 0)
 		(unit 1)
@@
 			)
 		)
-		(property "Value" "+5VA"
+		(property "Value" "+5VSB"
 			(at 266.7 167.64 0)
 			(effects
@@
 	)
 	(symbol
-		(lib_id "power:+5VA")
+		(lib_id "Hydra16:+5VSB")
 		(at 76.2 121.92 0)
 		(unit 1)
@@
 			)
 		)
-		(property "Value" "+5VA"
+		(property "Value" "+5VSB"
 			(at 76.2 118.11 0)
 			(effects
