File: board/Power.kicad_sch (KiCad schematic)
At the start: 20 parts, among them J37 PWR MODE, J7 Front Panel, J8 ATX-24, U36 DS1813-5, U78 74HC14, U79 74HC74

Commit message: V2.0: speaker headers, A/D bus fix, layout edits
- On-board speakers LS1/LS2 replaced by 2-pin headers J40 (SPEAKER L)
  and J41 (SPEAKER R) for external mini speakers: pin 1 speaker
  (through R30/R31), pin 2 GNDA; J18 still mutes them
- Connectors: a layout move had joined the A[0..15] and D[0..7] buses
  at two crossings (shorting A0-A7 to D0-D7); buses separated again,
  connectivity matches the previous commit
- Layout edits across the sheets (no other connectivity change)
- PCB updated from the schematic

Co-Authored-By: Claude Opus 5.5 <noreply@anthropic.com>
Other:
- title: Power: ATX, Front Panel, Reset, Soft Power -> Expansion Slots, SPI Headers and Port A
Changed lines of the file:
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@@
 	(paper "USLetter")
 	(title_block
-		(title "Power: ATX, Front Panel, Reset, Soft Power")
+		(title "Expansion Slots, SPI Headers and Port A")
 		(date "2026-10-06")
 		(rev "2.0D")
