File: board/WaitStates.kicad_sch (KiCad schematic)
At the start: 6 parts, among them U84 ATF22V10C-10PU, U87 ATF16V8C-10PU

Commit message: V2.0 rev 2.0D: clock stretching, OS ROM paging and review fixes
Bus timing:
- New GAL C (U88) generates PHI2/PHI1 and the 3.58 MHz sound clock from
  the 14.318 MHz master, replacing the U35 74F191 divider. J36 now selects
  7.16 or 3.58 MHz.
- Banked RAM, banked ROM and slot I/O ($FF20-$FFEF) get one extra PHI2-low
  period plus 0-3 extra PHI2-high periods set in $FFF5 (GAL D). This
  replaces the on-board RDY wait generator; cards can still pull RDY.
- Write strobes are now hold-time safe: PHI1 comes straight from GAL C
  and RWB_M straight from GAL B2.

Review fixes:
- OS ROM chip enable from a single-level decode, output enable from
  GAL B1; -55 part specified. Full 4K OS ROM paging via GAL G.
- Vector RAM writes only during PHI2; $FFF0-$FFFF no longer slowed.
- YM2151 /WR on RWB_M. U62 removed. RB0-RB7 pull-ups (RN5).
- Slot clocks driven through U56 and U34 with 33R series resistors.
- J38 enables in-system flashing of the banked ROMs.
- W65C22S/W65C51N, AS6C4008, DS1813-5 and CY7C192-25 values; R4 1k.
- J7 pin 8 no longer +5V; +5VA renamed +5VSB; serial handshake loop.
- Sheet titles and revisions, slot symbol pin fixes, and project symbol
  and footprint libraries so the project opens on another machine.

Co-Authored-By: Claude Opus 5.5 <noreply@anthropic.com>
Parts:
- R4: value 2.2k -> 1k
Connections:
- net CPU_RDY: no longer U84.23 (IO23)
- net GND: no longer U87.9 (I9)
- net ROM_A12: now reaches U87.13 (IO7)
- net N1: now reaches U84.22 (IO22)
- new net N0: U84.23 (IO23)
- new net RW6: U87.9 (I9)
- no-connect marks 11 -> 9
Other:
- note added: "CLOCK-STRETCH REGISTER $FFF5 (write-only, cleared by RESB) - U84 (GAL D) bits 1:0 banked RAM $8000-$9FFF bits 3:2 banked ROM $A000-$DFFF bits 5:4 slot I/O $FF20-$FFEF extra PHI2-high periods = 3 - value (69.8 ns each at 7.16 MHz) Reset leaves 3 extra periods everywhere. U88 (GAL C) also adds one PHI2-low period to every access in these regions, so addresses, bank registers and chip selects settle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"
- note removed: "WAIT-STATE REGISTER $FFF5 (write-only, cleared by RESB) - logic in U84 (GAL D) bits 1:0 banked RAM $8000-$9FFF waits = 3 - value bits 3:2 banked ROM $A000-$DFFF waits = 3 - value bits 5:4 I/O $FF20-$FFFF waits = 3 - value Reset leaves 3 waits everywhere. Main RAM, OS ROM and the VIA/ACIA never get waits. U84 drives CPU_RDY low only while stalling (R4 pulls it up; WAI still works). D1 lets a slot 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"
- title: Wait States and ROM Bank Gating (GALs) -> Clock-Stretch Control and OS ROM Paging (GALs)
Changed lines of the file:
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@@
 	(paper "A3")
 	(title_block
-		(title "Wait States and ROM Bank Gating (GALs)")
-		(date "2026-10-04")
-		(rev "2.0C")
+		(title "Clock-Stretch Control and OS ROM Paging (GALs)")
+		(date "2026-10-06")
+		(rev "2.0D")
 		(company "Data Tuning")
 		(comment 1 "Hydra 16")
 	)
-	(text "WAIT-STATE REGISTER  $FFF5  (write-only, cleared by RESB) - logic in U84 (GAL D)\n  bits 1:0  banked RAM  $8000-$9FFF     waits = 3 - value\n  bits 3:2  banked ROM  $A000-$DFFF     waits = 3 - value\n  bits 5:4  I/O $FF20-$FFFF              waits = 3 - value\nReset leaves 3 waits everywhere. Main RAM, OS ROM and the VIA/ACIA never get waits.\nU84 drives CPU_RDY low only while stalling (R4 pulls it up; WAI still works).\nD1 lets a slot card pulling bus RDY low stall the CPU; the CPU's WAI is not seen on bus RDY.\nU87 (GAL G): OS ROM bank lines W = RW for $E000-$EFFF, 0 for $F000-$FFFF."
+	(text "CLOCK-STRETCH REGISTER $FFF5 (write-only, cleared by RESB) - U84 (GAL D)\n  bits 1:0  banked RAM  $8000-$9FFF\n  bits 3:2  banked ROM  $A000-$DFFF\n  bits 5:4  slot I/O    $FF20-$FFEF       extra PHI2-high periods = 3 - value (69.8 ns each at 7.16 MHz)\nReset leaves 3 extra periods everywhere. U88 (GAL C) also adds one PHI2-low period to every access in\nthese regions, so addresses, bank registers and chip selects settle before PHI2 rises.\nMain RAM, OS ROM, VIA/ACIA and $FFF0-$FFFF are never stretched.\nCards can still pull RDY (D1) for longer waits; the CPU then repeats the cycle (one PHI2 strobe per repeat).\nU87 (GAL G): OS ROM paging. $E000-$EFFF = 4K page RW6..RW0, $F000-$FFFF = fixed page at ROM offset $1000."
 		(exclude_from_sim no)
 		(at 139.7 120.65 0)
@@
 	)
 	(no_connect
-		(at 91.44 66.04)
-	)
-	(no_connect
 		(at 88.9 165.1)
-	)
-	(no_connect
-		(at 88.9 162.56)
 	)
 	(no_connect
@@
 	(wire
 		(pts
+			(xy 163.83 93.98) (xy 166.37 93.98)
+		)
+		(stroke
+			(width 0)
+			(type default)
+		)
+	)
+	(wire
+		(pts
+			(xy 160.02 57.15) (xy 160.02 54.61)
+		)
+		(stroke
+			(width 0)
+			(type default)
+		)
+	)
+	(wire
+		(pts
+			(xy 63.5 157.48) (xy 60.96 157.48)
+		)
+		(stroke
+			(width 0)
+			(type default)
+		)
+	)
+	(wire
+		(pts
+			(xy 91.44 63.5) (xy 93.98 63.5)
+		)
+		(stroke
+			(width 0)
+			(type default)
+		)
+	)
+	(wire
+		(pts
+			(xy 160.02 64.77) (xy 160.02 67.31)
+		)
+		(stroke
+			(width 0)
+			(type default)
+		)
+	)
+	(wire
+		(pts
+			(xy 63.5 152.4) (xy 60.96 152.4)
+		)
+		(stroke
+			(width 0)
+			(type default)
+		)
+	)
+	(wire
+		(pts
+			(xy 63.5 160.02) (xy 60.96 160.02)
+		)
+		(stroke
+			(width 0)
+			(type default)
+		)
+	)
+	(wire
+		(pts
+			(xy 91.44 66.04) (xy 101.6 66.04)
+		)
+		(stroke
+			(width 0)
+			(type default)
+		)
+	)
+	(wire
+		(pts
 			(xy 63.5 167.64) (xy 60.96 167.64)
 		)
@@
 	(wire
 		(pts
-			(xy 163.83 93.98) (xy 166.37 93.98)
-		)
-		(stroke
-			(width 0)
-			(type default)
-		)
-	)
-	(wire
-		(pts
-			(xy 160.02 57.15) (xy 160.02 54.61)
-		)
-		(stroke
-			(width 0)
-			(type default)
-		)
-	)
-	(wire
-		(pts
-			(xy 63.5 157.48) (xy 60.96 157.48)
-		)
-		(stroke
-			(width 0)
-			(type default)
-		)
-	)
-	(wire
-		(pts
-			(xy 91.44 63.5) (xy 93.98 63.5)
-		)
-		(stroke
-			(width 0)
-			(type default)
-		)
-	)
-	(wire
-		(pts
-			(xy 160.02 64.77) (xy 160.02 67.31)
-		)
-		(stroke
-			(width 0)
-			(type default)
-		)
-	)
-	(wire
-		(pts
-			(xy 63.5 152.4) (xy 60.96 152.4)
-		)
-		(stroke
-			(width 0)
-			(type default)
-		)
-	)
-	(wire
-		(pts
-			(xy 63.5 160.02) (xy 60.96 160.02)
-		)
-		(stroke
-			(width 0)
-			(type default)
-		)
-	)
-	(global_label "CPU_RDY"
-		(shape bidirectional)
+			(xy 88.9 162.56) (xy 99.06 162.56)
+		)
+		(stroke
+			(width 0)
+			(type default)
+		)
+	)
+	(global_label "N0"
+		(shape output)
 		(at 93.98 63.5 0)
 		(fields_autoplaced yes)
@@
 				)
 				(justify right)
+				(hide yes)
+			)
+		)
+	)
+	(global_label "N1"
+		(shape output)
+		(at 101.6 66.04 0)
+		(fields_autoplaced yes)
+		(effects
+			(font
+				(size 1.27 1.27)
+			)
+			(justify left)
+		)
+		(property "Intersheetrefs" "${INTERSHEET_REFS}"
+			(at 101.6 66.04 0)
+			(effects
+				(font
+					(size 1.27 1.27)
+				)
+				(justify left)
+				(hide yes)
+			)
+		)
+	)
+	(global_label "RW6"
+		(shape input)
+		(at 60.96 167.64 180)
+		(fields_autoplaced yes)
+		(effects
+			(font
+				(size 1.27 1.27)
+			)
+			(justify right)
+		)
+		(property "Intersheetrefs" "${INTERSHEET_REFS}"
+			(at 60.96 167.64 180)
+			(effects
+				(font
+					(size 1.27 1.27)
+				)
+				(justify right)
+				(hide yes)
+			)
+		)
+	)
+	(global_label "ROM_A12"
+		(shape output)
+		(at 99.06 162.56 0)
+		(fields_autoplaced yes)
+		(effects
+			(font
+				(size 1.27 1.27)
+			)
+			(justify left)
+		)
+		(property "Intersheetrefs" "${INTERSHEET_REFS}"
+			(at 99.06 162.56 0)
+			(effects
+				(font
+					(size 1.27 1.27)
+				)
+				(justify left)
 				(hide yes)
 			)
@@
 	)
 	(symbol
-		(lib_id "power:GND")
-		(at 60.96 167.64 270)
-		(unit 1)
-		(exclude_from_sim no)
-		(in_bom yes)
-		(on_board yes)
-		(dnp no)
-		(property "Reference" "#PWR245"
-			(at 60.96 167.64 0)
-			(effects
-				(font
-					(size 1.27 1.27)
-				)
-				(hide yes)
-			)
-		)
-		(property "Value" "GND"
-			(at 55.88 167.64 0)
-			(effects
-				(font
-					(size 1.27 1.27)
-				)
-				(hide yes)
-			)
-		)
-		(property "Footprint" ""
-			(at 60.96 167.64 0)
-			(effects
-				(font
-					(size 1.27 1.27)
-				)
-				(hide yes)
-			)
-		)
-		(property "Datasheet" ""
-			(at 60.96 167.64 0)
-			(effects
-				(font
-					(size 1.27 1.27)
-				)
-				(hide yes)
-			)
-		)
-		(property "Description" "Power symbol creates a global label with name \"GND\""
-			(at 60.96 167.64 0)
-			(effects
-				(font
-					(size 1.27 1.27)
-				)
-				(hide yes)
-			)
-		)
-		(pin "1"
-		)
-		(instances
-			(project "hydra-16"
-				(path "/ef29fc71-3fec-48b5-8a1a-46bee537a98c/3d67b1b1-9a28-4462-8a4d-19765afeaafe"
-					(reference "#PWR245")
-					(unit 1)
-				)
-			)
-		)
-	)
-	(symbol
 		(lib_id "Device:D_Schottky")
 		(at 160.02 93.98 0)
@@
 			)
 		)
-		(property "Value" "2.2k"
+		(property "Value" "1k"
 			(at 163.83 62.23 0)
 			(effects
@@
 			)
 		)
-		(property "Datasheet" "GAL D - see board/PLDs/V2/GALD.PLD"
+		(property "Datasheet" "GAL D - clock-stretch register, see board/PLDs/V2/GALD.PLD"
 			(at 76.2 76.2 0)
 			(effects

Commit message: V2.0: split Support sheet, add stereo amplifier and on-board speakers
Support sheet reorganized (connectivity unchanged):
- Support.kicad_sch renamed to Power: ATX, front panel, reset, soft power, -5V
- Oscillators and their parts moved to Clocks (now US Ledger)
- Sound-chip decoupling and line-out parts moved to Sound
- VIA CB1/CB2/SPI pull-ups moved to Connectors
- Also includes minor schematic edits made before the reorganization

Audio output rework (Sound, now A3):
- U89 TDA2822M stereo amplifier on 9 V from U90 L7809 (fed by +12V)
- RV1 dual 10k log volume pot behind R26/R27 220k attenuators
- J18 moved from Connectors and now uses the switched TRS symbol:
  a plug lifts T/R off TN/RN and mutes the on-board speakers
- LS1/LS2 8 ohm mini speakers through R30/R31 (15R 0.5 W)
- New footprint Speaker_D32mm_P15.24mm_P17.50mm (two pad pairs, fits
  Adafruit 1898 or Kitronik 3316)
- J39 line-out header (LINE_L, LINE_R, GNDA)
- R18 stays the single GNDA-GND tie, to sit at U89 pin 4
- TDA2822M symbol added to hydra16.kicad_sym

Co-Authored-By: Claude Opus 5.5 <noreply@anthropic.com>
Other:
- moved on the sheet: R4
Changed lines of the file:
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@@
 		)
+	)
+	(junction
+		(at 167.64 93.98)
+		(diameter 0)
+		(color 0 0 0 0)
 	)
 	(no_connect
@@
 	(wire
 		(pts
+			(xy 91.44 66.04) (xy 101.6 66.04)
+		)
+		(stroke
+			(width 0)
+			(type default)
+		)
+	)
+	(wire
+		(pts
+			(xy 63.5 167.64) (xy 60.96 167.64)
+		)
+		(stroke
+			(width 0)
+			(type default)
+		)
+	)
+	(wire
+		(pts
 			(xy 60.96 76.2) (xy 58.42 76.2)
 		)
@@
 	(wire
 		(pts
+			(xy 88.9 162.56) (xy 99.06 162.56)
+		)
+		(stroke
+			(width 0)
+			(type default)
+		)
+	)
+	(wire
+		(pts
 			(xy 76.2 55.88) (xy 76.2 53.34)
 		)
@@
 	(wire
 		(pts
+			(xy 167.64 87.63) (xy 167.64 93.98)
+		)
+		(stroke
+			(width 0)
+			(type default)
+		)
+	)
+	(wire
+		(pts
 			(xy 60.96 86.36) (xy 58.42 86.36)
 		)
@@
 	(wire
 		(pts
-			(xy 163.83 93.98) (xy 166.37 93.98)
-		)
-		(stroke
-			(width 0)
-			(type default)
-		)
-	)
-	(wire
-		(pts
-			(xy 160.02 57.15) (xy 160.02 54.61)
+			(xy 163.83 93.98) (xy 167.64 93.98)
+		)
+		(stroke
+			(width 0)
+			(type default)
+		)
+	)
+	(wire
+		(pts
+			(xy 167.64 80.01) (xy 167.64 77.47)
 		)
 		(stroke
@@
 	(wire
 		(pts
-			(xy 160.02 64.77) (xy 160.02 67.31)
+			(xy 167.64 93.98) (xy 173.99 93.98)
 		)
 		(stroke
@@
 		(pts
 			(xy 63.5 160.02) (xy 60.96 160.02)
-		)
-		(stroke
-			(width 0)
-			(type default)
-		)
-	)
-	(wire
-		(pts
-			(xy 91.44 66.04) (xy 101.6 66.04)
-		)
-		(stroke
-			(width 0)
-			(type default)
-		)
-	)
-	(wire
-		(pts
-			(xy 63.5 167.64) (xy 60.96 167.64)
-		)
-		(stroke
-			(width 0)
-			(type default)
-		)
-	)
-	(wire
-		(pts
-			(xy 88.9 162.56) (xy 99.06 162.56)
 		)
 		(stroke
@@
 		)
 	)
-	(global_label "CPU_RDY"
-		(shape bidirectional)
-		(at 160.02 67.31 270)
-		(fields_autoplaced yes)
-		(effects
-			(font
-				(size 1.27 1.27)
-			)
-			(justify right)
-		)
-		(property "Intersheetrefs" "${INTERSHEET_REFS}"
-			(at 160.02 67.31 270)
-			(effects
-				(font
-					(size 1.27 1.27)
-				)
-				(justify right)
-				(hide yes)
-			)
-		)
-	)
 	(global_label "W3"
 		(shape output)
@@
 		)
 	)
+	(global_label "N1"
+		(shape output)
+		(at 101.6 66.04 0)
+		(fields_autoplaced yes)
+		(effects
+			(font
+				(size 1.27 1.27)
+			)
+			(justify left)
+		)
+		(property "Intersheetrefs" "${INTERSHEET_REFS}"
+			(at 101.6 66.04 0)
+			(effects
+				(font
+					(size 1.27 1.27)
+				)
+				(justify left)
+				(hide yes)
+			)
+		)
+	)
 	(global_label "RW0"
 		(shape input)
@@
 				)
 				(justify right)
+				(hide yes)
+			)
+		)
+	)
+	(global_label "ROM_A12"
+		(shape output)
+		(at 99.06 162.56 0)
+		(fields_autoplaced yes)
+		(effects
+			(font
+				(size 1.27 1.27)
+			)
+			(justify left)
+		)
+		(property "Intersheetrefs" "${INTERSHEET_REFS}"
+			(at 99.06 162.56 0)
+			(effects
+				(font
+					(size 1.27 1.27)
+				)
+				(justify left)
 				(hide yes)
 			)
@@
 		)
 	)
+	(global_label "RW6"
+		(shape input)
+		(at 60.96 167.64 180)
+		(fields_autoplaced yes)
+		(effects
+			(font
+				(size 1.27 1.27)
+			)
+			(justify right)
+		)
+		(property "Intersheetrefs" "${INTERSHEET_REFS}"
+			(at 60.96 167.64 180)
+			(effects
+				(font
+					(size 1.27 1.27)
+				)
+				(justify right)
+				(hide yes)
+			)
+		)
+	)
 	(global_label "RW4"
 		(shape input)
@@
 	(global_label "CPU_RDY"
 		(shape bidirectional)
-		(at 166.37 93.98 0)
+		(at 173.99 93.98 0)
 		(fields_autoplaced yes)
 		(effects
@@
 		)
 		(property "Intersheetrefs" "${INTERSHEET_REFS}"
-			(at 166.37 93.98 0)
+			(at 173.99 93.98 0)
 			(effects
 				(font
@@
 				)
 				(justify right)
-				(hide yes)
-			)
-		)
-	)
-	(global_label "N1"
-		(shape output)
-		(at 101.6 66.04 0)
-		(fields_autoplaced yes)
-		(effects
-			(font
-				(size 1.27 1.27)
-			)
-			(justify left)
-		)
-		(property "Intersheetrefs" "${INTERSHEET_REFS}"
-			(at 101.6 66.04 0)
-			(effects
-				(font
-					(size 1.27 1.27)
-				)
-				(justify left)
-				(hide yes)
-			)
-		)
-	)
-	(global_label "RW6"
-		(shape input)
-		(at 60.96 167.64 180)
-		(fields_autoplaced yes)
-		(effects
-			(font
-				(size 1.27 1.27)
-			)
-			(justify right)
-		)
-		(property "Intersheetrefs" "${INTERSHEET_REFS}"
-			(at 60.96 167.64 180)
-			(effects
-				(font
-					(size 1.27 1.27)
-				)
-				(justify right)
-				(hide yes)
-			)
-		)
-	)
-	(global_label "ROM_A12"
-		(shape output)
-		(at 99.06 162.56 0)
-		(fields_autoplaced yes)
-		(effects
-			(font
-				(size 1.27 1.27)
-			)
-			(justify left)
-		)
-		(property "Intersheetrefs" "${INTERSHEET_REFS}"
-			(at 99.06 162.56 0)
-			(effects
-				(font
-					(size 1.27 1.27)
-				)
-				(justify left)
 				(hide yes)
 			)
@@
 	(symbol
 		(lib_id "power:+5V")
-		(at 160.02 54.61 0)
+		(at 167.64 77.47 0)
 		(unit 1)
 		(exclude_from_sim no)
@@
 		(dnp no)
 		(property "Reference" "#PWR249"
-			(at 160.02 54.61 0)
+			(at 167.64 77.47 0)
 			(effects
 				(font
@@
 		)
 		(property "Value" "+5V"
-			(at 160.02 50.8 0)
+			(at 167.64 73.66 0)
 			(effects
 				(font
@@
 		)
 		(property "Footprint" ""
-			(at 160.02 54.61 0)
+			(at 167.64 77.47 0)
 			(effects
 				(font
@@
 		)
 		(property "Datasheet" ""
-			(at 160.02 54.61 0)
+			(at 167.64 77.47 0)
 			(effects
 				(font
@@
 		)
 		(property "Description" "Power symbol creates a global label with name \"+5V\""
-			(at 160.02 54.61 0)
+			(at 167.64 77.47 0)
 			(effects
 				(font
@@
 	(symbol
 		(lib_id "Device:R")
-		(at 160.02 60.96 0)
+		(at 167.64 83.82 0)
 		(unit 1)
 		(exclude_from_sim no)
@@
 		(dnp no)
 		(property "Reference" "R4"
-			(at 163.83 59.69 0)
+			(at 171.45 82.55 0)
 			(effects
 				(font
@@
 		)
 		(property "Value" "1k"
-			(at 163.83 62.23 0)
+			(at 171.45 85.09 0)
 			(effects
 				(font
@@
 		)
 		(property "Footprint" "Resistor_THT:R_Axial_DIN0204_L3.6mm_D1.6mm_P5.08mm_Horizontal"
-			(at 160.02 60.96 0)
+			(at 167.64 83.82 0)
 			(effects
 				(font
@@
 		)
 		(property "Datasheet" ""
-			(at 160.02 60.96 0)
+			(at 167.64 83.82 0)
 			(effects
 				(font
@@
 		)
 		(property "Description" ""
-			(at 160.02 60.96 0)
-			(effects
-				(font
+			(at 167.64 83.82 0)
+			(effects
+				(font
