File: board/MemoryDaughterCard/MemDaughterCard.kicad_sch (KiCad schematic)
At the start: 13 parts, among them IC1 HM628512LP-7, IC2 HM628512LP-7, IC3 HM628512LP-7, IC4 HM628512LP-7, J1 Conn_01x32, J2 Conn_01x24, J3 Conn_02x15_Odd_Even, U1 74LS139

Commit message: Board V1.1G
Other:
- moved on the sheet: C1, C2, C3, C4, C5, IC1, IC2, IC3, IC4, J1, J2, J3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
