File: board/MemoryDaughterCard/MemDaughterCard_SurfaceMount.kicad_sch (KiCad schematic)
At the start: 18 parts, among them IC1 HM628512LFP-7, IC2 HM628512LFP-7, IC3 HM628512LFP-7, IC4 HM628512LFP-7, IC5 HM628512LFP-7, IC6 HM628512LFP-7, IC7 HM628512LFP-7, IC8 HM628512LFP-7, J1 Conn_01x32, J2 Conn_01x24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

Commit message: Board V1.1G
Parts:
- renumbered C6 to C4, IC4 to IC1, IC1 to IC2, IC2 to IC3, IC3 to IC4
Changed lines of the file:
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@@
 (kicad_sch
-	(version 20231120)
+	(version 20250114)
 	(generator "eeschema")
-	(generator_version "8.0")
+	(generator_version "9.0")
 	(paper "B")
 	(junction
@@
 	)
 	(junction
-		(at 110.49 152.4)
+		(at 279.4 160.02)
 		(diameter 0)
 		(color 0 0 0 0)
 	)
 	(junction
-		(at 261.62 92.71)
+		(at 110.49 152.4)
 		(diameter 0)
 		(color 0 0 0 0)
 	)
 	(junction
-		(at 279.4 161.29)
+		(at 261.62 92.71)
 		(diameter 0)
 		(color 0 0 0 0)
@@
 	)
 	(junction
+		(at 232.41 160.02)
+		(diameter 0)
+		(color 0 0 0 0)
+	)
+	(junction
 		(at 289.56 130.81)
 		(diameter 0)
@@
 	)
 	(junction
-		(at 232.41 161.29)
-		(diameter 0)
-		(color 0 0 0 0)
-	)
-	(junction
 		(at 95.25 48.26)
 		(diameter 0)
@@
 	)
 	(junction
-		(at 224.79 161.29)
+		(at 289.56 115.57)
 		(diameter 0)
 		(color 0 0 0 0)
 	)
 	(junction
-		(at 289.56 115.57)
+		(at 177.8 152.4)
 		(diameter 0)
 		(color 0 0 0 0)
 	)
 	(junction
-		(at 177.8 152.4)
+		(at 224.79 160.02)
 		(diameter 0)
 		(color 0 0 0 0)
@@
 	(wire
 		(pts
-			(xy 279.4 161.29) (xy 279.4 160.02)
+			(xy 279.4 160.02) (xy 279.4 171.45)
 		)
 		(stroke
@@
 	(wire
 		(pts
+			(xy 232.41 160.02) (xy 232.41 161.29)
+		)
+		(stroke
+			(width 0)
+			(type default)
+		)
+	)
+	(wire
+		(pts
 			(xy 99.06 66.04) (xy 92.71 66.04)
 		)
@@
 	(wire
 		(pts
-			(xy 224.79 161.29) (xy 232.41 161.29)
+			(xy 224.79 160.02) (xy 232.41 160.02)
 		)
 		(stroke
@@
 	(wire
 		(pts
-			(xy 111.76 161.29) (xy 111.76 93.98)
+			(xy 111.76 160.02) (xy 111.76 93.98)
 		)
 		(stroke
@@
 	(wire
 		(pts
+			(xy 224.79 160.02) (xy 224.79 171.45)
+		)
+		(stroke
+			(width 0)
+			(type default)
+		)
+	)
+	(wire
+		(pts
 			(xy 95.25 21.59) (xy 95.25 45.72)
 		)
@@
 	(wire
 		(pts
-			(xy 224.79 161.29) (xy 111.76 161.29)
+			(xy 224.79 160.02) (xy 111.76 160.02)
 		)
 		(stroke
@@
 	(wire
 		(pts
-			(xy 232.41 161.29) (xy 279.4 161.29)
+			(xy 232.41 160.02) (xy 279.4 160.02)
 		)
 		(stroke
@@
 	(wire
 		(pts
-			(xy 279.4 171.45) (xy 279.4 161.29)
-		)
-		(stroke
-			(width 0)
-			(type default)
-		)
-	)
-	(wire
-		(pts
 			(xy 149.86 57.15) (xy 149.86 59.69)
 		)
@@
 	(wire
 		(pts
-			(xy 224.79 161.29) (xy 224.79 171.45)
-		)
-		(stroke
-			(width 0)
-			(type default)
-		)
-	)
-	(wire
-		(pts
 			(xy 289.56 128.27) (xy 289.56 130.81)
 		)
@@
 		(dnp no)
 		(fields_autoplaced yes)
-		(property "Reference" "C6"
+		(property "Reference" "C4"
 			(at 344.17 161.2962 0)
 			(effects
@@
 			(project "MemDaughterCard_SurfaceMount"
 				(path "/ef29fc71-3fec-48b5-8a1a-46bee537a98c"
-					(reference "C6")
+					(reference "C4")
 					(unit 1)
 				)
@@
 		(dnp no)
 		(fields_autoplaced yes)
-		(property "Reference" "IC4"
+		(property "Reference" "IC1"
 			(at 81.28 96.52 0)
 			(effects
@@
 			(project ""
 				(path "/ef29fc71-3fec-48b5-8a1a-46bee537a98c"
-					(reference "IC4")
+					(reference "IC1")
 					(unit 1)
 				)
@@
 		(dnp no)
 		(fields_autoplaced yes)
-		(property "Reference" "IC1"
+		(property "Reference" "IC2"
 			(at 135.89 96.52 0)
 			(effects
@@
 			(project "MemDaughterCard_SurfaceMount"
 				(path "/ef29fc71-3fec-48b5-8a1a-46bee537a98c"
-					(reference "IC1")
+					(reference "IC2")
 					(unit 1)
 				)
@@
 		(dnp no)
 		(fields_autoplaced yes)
-		(property "Reference" "IC3"
+		(property "Reference" "IC4"
 			(at 247.65 96.52 0)
 			(effects
@@
 			(project "MemDaughterCard_SurfaceMount"
 				(path "/ef29fc71-3fec-48b5-8a1a-46bee537a98c"
-					(reference "IC3")
+					(reference "IC4")
 					(unit 1)
 				)
@@
 		(dnp no)
 		(fields_autoplaced yes)
-		(property "Reference" "IC2"
+		(property "Reference" "IC3"
 			(at 193.04 96.52 0)
 			(effects
@@
 			(project "MemDaughterCard_SurfaceMount"
 				(path "/ef29fc71-3fec-48b5-8a1a-46bee537a98c"
-					(reference "IC2")
+					(reference "IC3")
 					(unit 1)
 				)
@@
 		)
 	)
+	(embedded_fonts no)
 )
