File: board/MemoryDaughterCard/MemDaughterCard_SurfaceMount.kicad_pcb (KiCad board)
At the start: 2 copper layers, 88.9 x 67.3 mm, 18 parts, among them IC1 HM628512LFP-7, IC2 HM628512LFP-7, IC3 HM628512LFP-7, IC4 HM628512LFP-7, IC5 HM628512LFP-7, IC6 HM628512LFP-7, IC7 HM628512LFP-7, IC8 HM628512LFP-7, J1 Conn_01x32, J2 Conn_01x24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

Commit message: Minor updates post board fab
Routing:
- net Net-(IC8-~{CS}): track 53.5 -> 50.7 mm
- net D6: track 172.4 -> 174.5 mm
- net T2: track 193.6 -> 194.1 mm
