File: board/MemoryDaughterCard/MemDaughterCard_SurfaceMount_Edge.kicad_sch (KiCad schematic)
At the start: 18 parts, among them IC1 HM628512LFP-7, IC2 HM628512LFP-7, IC3 HM628512LFP-7, IC4 HM628512LFP-7, IC5 HM628512LFP-7, IC6 HM628512LFP-7, IC7 HM628512LFP-7, IC8 HM628512LFP-7, J1 Conn_01x32, J2 Conn_01x24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

Commit message: V2.0 updates and new hydra breakout and counter cards.
Parts:
- removed J1: Conn_01x32, Connector_PinHeader_2.54mm:PinHeader_1x32_P2.54mm_Vertical, symbol Connector_Generic:Conn_01x32
- removed J2: Conn_01x24, Connector_PinHeader_2.54mm:PinHeader_1x24_P2.54mm_Vertical, symbol Connector_Generic:Conn_01x24
- removed J3: Conn_02x15_Odd_Even, Connector_PinHeader_2.54mm:PinHeader_2x15_P2.54mm_Vertical, symbol Connector_Generic:Conn_02x15_Odd_Even
- removed J4: Conn_01x15_Pin, Connector_PinHeader_2.54mm:PinHeader_1x15_P2.54mm_Vertical, symbol Connector:Conn_01x15_Pin
- added C1, C2, C6, C8: 104, Capacitor_THT:C_Disc_D5.0mm_W2.5mm_P5.00mm, symbol Device:C_Small
- added J5: Conn_02x18_Top_Bottom, CustomLibrary:Bus_Hydra_Mem, symbol Connector_Generic:Conn_02x18_Top_Bottom
- C3: renamed from C4; value .1uF -> 104
- C4: renamed from C3; value .1uF -> 104
- C5: renamed from C1; value .1uF -> 104
- C7: renamed from C2; value .1uF -> 104
- C9: renamed from C5; value .1uF -> 104
Connections:
- net !RWB: now also J5.30 (Pin_30)
- net +5v: now also C1.1, C2.1, C6.1, C8.1, J5.1 (Pin_1)
- net A0: now also J5.2 (Pin_2)
- net A1: now also J5.3 (Pin_3)
- net A10: now also J5.12 (Pin_12)
- net A11: now also J5.13 (Pin_13)
- net A12: now also J5.14 (Pin_14)
- net A2: now also J5.4 (Pin_4)
- net A3: now also J5.5 (Pin_5)
- net A4: now also J5.6 (Pin_6)
- net A5: now also J5.7 (Pin_7)
- net A6: now also J5.8 (Pin_8)
- net A7: now also J5.9 (Pin_9)
- net A8: now also J5.10 (Pin_10)
- net A9: now also J5.11 (Pin_11)
- net D0: now also J5.20 (Pin_20)
- net D1: now also J5.21 (Pin_21)
- net D2: now also J5.22 (Pin_22)
- net D3: now also J5.23 (Pin_23)
- net D4: now also J5.24 (Pin_24)
- net D5: now also J5.25 (Pin_25)
- net D6: now also J5.26 (Pin_26)
- net D7: now also J5.27 (Pin_27)
- net GND: now also C1.2, C2.2, C6.2, C8.2, J5.19 (Pin_19), J5.28 (Pin_28)
- net RAMB0: now also J5.15 (Pin_15)
- net RAMB1: now also J5.16 (Pin_16)
- net RAMB2: now also J5.17 (Pin_17)
- net RAMB3: now also J5.18 (Pin_18)
- net RWB: now also J5.29 (Pin_29)
- net T0: now also J5.33 (Pin_33)
- net T1: now also J5.34 (Pin_34)
- net T2: now also J5.35 (Pin_35)
- net T3: now also J5.36 (Pin_36)
- net nSel1: now reaches U1.15 (~{EN})
- net nSel1: now also J5.32 (Pin_32)
- net nSel0: now reaches U1.1 (~{EN})
- net nSel0: now also J5.31 (Pin_31)
Other:
- moved on the sheet: C3, C4, C5, C7, C9, IC1, IC2, IC3, IC4, IC5, IC6, IC7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
