File: board/CycleCounterCard/counter-card/counter-card.kicad_pcb (KiCad board)
At the start: 6 copper layers, 106.7 x 105.4 mm, 33 parts, among them J1 Bus_Hydra_8bit, J2 74F86, J3 74F86, J4 74F86, J5 74F86, J7 A B, U1 74F191, U10 74F191, U11 74F191, U12 74F573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

Commit message: Counter card updated to 4-layer to make production simpler and cheaper.  Production V1 model.
Parts:
- I/O Port: renamed from J7
Connections:
- J3 pad 2: Q9 -> Q6
- J3 pad 4: Q17 -> Q15
- J4 pad 5: Q6 -> Q9
- J5 pad 10: Q15 -> Q17
Routing:
- net GND: track 18.7 -> 701.5 mm, vias 3 -> 0
- net +5V: track 13.4 -> 567.9 mm, vias 2 -> 0
- net Q15: track 118.3 -> 59.8 mm
- net Q17: track 139.2 -> 86.8 mm
- net Q6: track 113.7 -> 63.2 mm, vias 0 -> 1
- net Q5: track 128.8 -> 167.5 mm, vias 1 -> 0
- net Q2: track 119.3 -> 157.1 mm, vias 1 -> 0
- net Q8: track 125.7 -> 159.5 mm, vias 1 -> 0
- net Q0: track 113.4 -> 146.3 mm, vias 1 -> 0
- net Q27: track 73.5 -> 47.5 mm
- net Q7: track 114.0 -> 137.2 mm
- net Q22: track 122.6 -> 99.7 mm, vias 1 -> 0
- net Q19: track 92.2 -> 72.5 mm, vias 0 -> 1
- net OE7_S: track 78.7 -> 96.9 mm, vias 1 -> 0
- net OE3_S: track 102.4 -> 86.4 mm, vias 1 -> 0
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- removed copper zone on In1.Cu, net +5V
- removed copper zone on In4.Cu, net GND
Other:
- copper layers 6 -> 4
- board text removed: "I/O Port"
