File: board/CycleCounterCard/counter-card/counter-card.kicad_sch (KiCad schematic)
At the start: 16 parts, among them J7 Conn_01x03_Pin, U10 74F191, U11 74F191, U12 74F573, U14 74F191, U15 74F191, U16 74F191, U17 74F191, U18 74F573, U19 74F573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

Commit message: Counter card updated to 4-layer to make production simpler and cheaper.  Production V1 model.
Parts:
- renumbered J7 to IOPortSel
Changed lines of the file:
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@@
 		(dnp no)
 		(fields_autoplaced yes)
-		(property "Reference" "J7"
+		(property "Reference" "IOPortSel"
 			(at 36.83 175.2599 0)
 			(effects
@@
 			(project ""
 				(path "/57d288fb-0573-473e-905d-e34f81a4c3e2"
-					(reference "J7")
+					(reference "IOPortSel")
 					(unit 1)
 				)
