File: board/CycleCounterCard/counter-card/counter-card.kicad_sch (KiCad schematic)
At the start: 16 parts, among them U10 74F191, U11 74F191, U12 74F573, U14 74F191, U15 74F191, U16 74F191, U17 74F191, U18 74F573, U19 74F573, U24 74F02, U26 74F573, U27 74F00, U3 74F138, U8 74F191, U9 74F191

Commit message: V2.0: wait states, GAL glue logic, serial clock and review fixes
Main board schematic:
- Replace the T4-T7 clock divider with RDY wait states. Fixed 7.16 MHz
  CPU clock; J36 selects 3.58 MHz for Rockwell parts. Waits are set per
  region through the write-only register at $FFF5 (reset = 3 waits).
- Move address decode, strobes, the wait-state generator, the IRQ
  encoder/latch/vector mux, ROM bank gating and DMA sync into seven GALs
  (U81-U86 ATF22V10C, U87 ATF16V8C), removing 29 ICs. CUPL sources,
  JEDECs and notes are in board/PLDs/V2.
- 1.8432 MHz serial clock, soft-power latch, -5V regulator, bulk caps,
  pull-ups, audio coupling/decoupling, GNDA tie, read-only Z register
  and other design-review fixes.
- New WaitStates and Support sheets; project symbol library
  hydra16.kicad_sym with sym-lib-table.

PCB updated from the schematic. Includes pending changes to the counter,
bus breakout and memory daughter card projects.

Firmware:
- Remove S_REGISTER; T/U/V/W now at $FFF0-$FFF3 to match the hardware.
- Add math.s and sound.s (included by os_main.s).
- Rebuild the 65C02 ROM image.

Co-Authored-By: Claude Opus 5.5 <noreply@anthropic.com>
Parts:
- added C1, C2, C3, C4, C5, C6, C7, C8: 104, Capacitor_THT:C_Disc_D5.0mm_W2.5mm_P5.00mm, symbol Device:C
- added J6: Conn_02x03_Odd_Even, Connector_PinHeader_2.54mm:PinHeader_2x03_P2.54mm_Vertical, symbol Connector_Generic:Conn_02x03_Odd_Even
- renumbered IOPortSel to IOPortSel1
Connections:
- net +5V: now also C1.2, C2.2, C3.2, C4.2, C5.2, C6.2, C7.2, C8.2
- net GND: now also C1.1, C2.1, C3.1, C4.1, C5.1, C6.1, C7.1, C8.1
- net NMIB: now also J6.6 (Pin_6); no longer U27.3
- new net: J6.1 (Pin_1), J6.3 (Pin_3), J6.5 (Pin_5), U27.3
- new net IRQA: J6.2 (Pin_2)
- new net IRQB: J6.4 (Pin_4)
Other:
- moved on the sheet: IOPortSel1
