File: board/HydraBusBreakoutCard/HydraBusBreakoutCard.kicad_pcb (KiCad board)
At the start: 4 copper layers, 163.4 x 105.4 mm, 33 parts, among them J1 Bus_Hydra_8bit, J10 I2C, J11 Power, J17 Conn_02x40_Odd_Even, J18 Conn_02x40_Odd_Even, J19 Conn_02x40_Odd_Even, J2 Data Bus, J20 Conn_02x40_Odd_Even, J21 Conn_02x40_Odd_Even, J22 Conn_02x40_Odd_Even, J23 Conn_02x40_Odd_Even, J24 Conn_02x40_Odd_Even, J25 Conn_02x40_Odd_Even, J26 Conn_02x40_Odd_Even, J27 Conn_02x40_Odd_Even, J28 Conn_02x40_Odd_Even, J29 Conn_02x40_Odd_Even, J3 Address Bus, J30 Conn_02x40_Odd_Even, J31 Conn_02x40_Odd_Even, J32 Conn_02x40_Odd_Even, J33 Conn_02x40_Odd_Even, J34 Conn_02x40_Odd_Even, J4 SPI, J5 Interrupts & I/O, J6 Clocks, J7 Bus Control, J8 Reset, J9 Audio

Commit message: V2.0: wait states, GAL glue logic, serial clock and review fixes
Main board schematic:
- Replace the T4-T7 clock divider with RDY wait states. Fixed 7.16 MHz
  CPU clock; J36 selects 3.58 MHz for Rockwell parts. Waits are set per
  region through the write-only register at $FFF5 (reset = 3 waits).
- Move address decode, strobes, the wait-state generator, the IRQ
  encoder/latch/vector mux, ROM bank gating and DMA sync into seven GALs
  (U81-U86 ATF22V10C, U87 ATF16V8C), removing 29 ICs. CUPL sources,
  JEDECs and notes are in board/PLDs/V2.
- 1.8432 MHz serial clock, soft-power latch, -5V regulator, bulk caps,
  pull-ups, audio coupling/decoupling, GNDA tie, read-only Z register
  and other design-review fixes.
- New WaitStates and Support sheets; project symbol library
  hydra16.kicad_sym with sym-lib-table.

PCB updated from the schematic. Includes pending changes to the counter,
bus breakout and memory daughter card projects.

Firmware:
- Remove S_REGISTER; T/U/V/W now at $FFF0-$FFF3 to match the hardware.
- Add math.s and sound.s (included by os_main.s).
- Rebuild the 65C02 ROM image.

Co-Authored-By: Claude Opus 5.5 <noreply@anthropic.com>
Parts:
- H1, H3, H4: value MountingHole_3.2mm_M3 -> MountingHole
- H2: value MountingHole_3.2mm_M3_ISO7380_Pad_TopBottom -> MountingHole_Pad
- moved J3 16.9 mm to (204.5, 105.4)
- moved J2 9.67 mm to (204.5, 128.3)
- moved H4 0.25 mm to (247.3, 43.3)
Connections:
- J17 pad 78: unconnected-(J17-Pin_78-Pad78) -> GND
- J17 pad 79: GND -> +5V
- J18 pad 77: unconnected-(J18-Pin_77-Pad77) -> GND
- J18 pad 78: unconnected-(J18-Pin_78-Pad78) -> GND
- J19 pad 77: unconnected-(J19-Pin_77-Pad77) -> GND
- J19 pad 78: unconnected-(J19-Pin_78-Pad78) -> GND
- J20 pad 77: unconnected-(J20-Pin_77-Pad77) -> GND
- J20 pad 78: unconnected-(J20-Pin_78-Pad78) -> GND
- J21 pad 77: unconnected-(J21-Pin_77-Pad77) -> GND
- J21 pad 78: unconnected-(J21-Pin_78-Pad78) -> GND
- J22 pad 77: unconnected-(J22-Pin_77-Pad77) -> GND
- J22 pad 78: unconnected-(J22-Pin_78-Pad78) -> GND
- J23 pad 77: unconnected-(J23-Pin_77-Pad77) -> GND
- J23 pad 78: unconnected-(J23-Pin_78-Pad78) -> GND
- J24 pad 77: unconnected-(J24-Pin_77-Pad77) -> GND
- J24 pad 78: unconnected-(J24-Pin_78-Pad78) -> GND
- J25 pad 77: unconnected-(J25-Pin_77-Pad77) -> GND
- J25 pad 78: unconnected-(J25-Pin_78-Pad78) -> GND
- J26 pad 77: unconnected-(J26-Pin_77-Pad77) -> GND
- J26 pad 78: unconnected-(J26-Pin_78-Pad78) -> GND
- J27 pad 77: unconnected-(J27-Pin_77-Pad77) -> GND
- J27 pad 78: unconnected-(J27-Pin_78-Pad78) -> GND
- J28 pad 77: unconnected-(J28-Pin_77-Pad77) -> GND
- J28 pad 78: unconnected-(J28-Pin_78-Pad78) -> GND
- J29 pad 77: unconnected-(J29-Pin_77-Pad77) -> GND
- J29 pad 78: unconnected-(J29-Pin_78-Pad78) -> GND
- J30 pad 77: unconnected-(J30-Pin_77-Pad77) -> GND
- J30 pad 78: unconnected-(J30-Pin_78-Pad78) -> GND
- J31 pad 77: unconnected-(J31-Pin_77-Pad77) -> GND
- J31 pad 78: unconnected-(J31-Pin_78-Pad78) -> GND
- J32 pad 77: unconnected-(J32-Pin_77-Pad77) -> GND
- J32 pad 78: unconnected-(J32-Pin_78-Pad78) -> GND
- J33 pad 77: unconnected-(J33-Pin_77-Pad77) -> GND
- J33 pad 78: unconnected-(J33-Pin_78-Pad78) -> GND
- J34 pad 77: unconnected-(J34-Pin_77-Pad77) -> GND
- J34 pad 78: unconnected-(J34-Pin_78-Pad78) -> GND
Routing:
- net Net-(J1-DB0): track 46.2 -> 63.4 mm
- net Net-(J1-A00): track 116.4 -> 99.5 mm
- net Net-(J1-A01): track 111.4 -> 95.4 mm
- net Net-(J1-A07): track 86.1 -> 70.3 mm, vias 1 -> 0
- net Net-(J1-A12): track 65.5 -> 49.9 mm, vias 1 -> 0
- net Net-(J1-A08): track 81.8 -> 66.2 mm
- net Net-(J1-A11): track 69.5 -> 54.0 mm, vias 1 -> 0
- net Net-(J1-DB4): track 42.5 -> 27.0 mm, vias 0 -> 1
- net Net-(J1-A03): track 102.3 -> 86.8 mm, vias 1 -> 0
- net Net-(J1-A09): track 77.7 -> 62.2 mm
- net Net-(J1-A02): track 106.1 -> 90.8 mm
- net Net-(J1-A14): track 57.3 -> 42.2 mm
- net Net-(J1-DB3): track 43.6 -> 28.4 mm, vias 0 -> 1
- net Net-(J1-A10): track 73.0 -> 58.0 mm
- net Net-(J1-A04): track 97.6 -> 82.6 mm
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Other:
- board size 163.4 x 105.4 mm -> 160.9 x 105.4 mm
- board text added: "Hydra Prototyping and Breakout Card V1.1"
