File: board/HydraBusBreakoutCard/HydraBusBreakoutCard.kicad_sch (KiCad schematic)
At the start: 29 parts, among them J1 Bus_Hydra_8bit, J10 I2C, J11 Power, J17 Conn_02x40_Odd_Even, J18 Conn_02x40_Odd_Even, J19 Conn_02x40_Odd_Even, J2 Data Bus, J20 Conn_02x40_Odd_Even, J21 Conn_02x40_Odd_Even, J22 Conn_02x40_Odd_Even, J23 Conn_02x40_Odd_Even, J24 Conn_02x40_Odd_Even, J25 Conn_02x40_Odd_Even, J26 Conn_02x40_Odd_Even, J27 Conn_02x40_Odd_Even, J28 Conn_02x40_Odd_Even, J29 Conn_02x40_Odd_Even, J3 Address Bus, J30 Conn_02x40_Odd_Even, J31 Conn_02x40_Odd_Even, J32 Conn_02x40_Odd_Even, J33 Conn_02x40_Odd_Even, J34 Conn_02x40_Odd_Even, J4 SPI, J5 Interrupts & I/O, J6 Clocks, J7 Bus Control, J8 Reset, J9 Audio

Commit message: V2.0: wait states, GAL glue logic, serial clock and review fixes
Main board schematic:
- Replace the T4-T7 clock divider with RDY wait states. Fixed 7.16 MHz
  CPU clock; J36 selects 3.58 MHz for Rockwell parts. Waits are set per
  region through the write-only register at $FFF5 (reset = 3 waits).
- Move address decode, strobes, the wait-state generator, the IRQ
  encoder/latch/vector mux, ROM bank gating and DMA sync into seven GALs
  (U81-U86 ATF22V10C, U87 ATF16V8C), removing 29 ICs. CUPL sources,
  JEDECs and notes are in board/PLDs/V2.
- 1.8432 MHz serial clock, soft-power latch, -5V regulator, bulk caps,
  pull-ups, audio coupling/decoupling, GNDA tie, read-only Z register
  and other design-review fixes.
- New WaitStates and Support sheets; project symbol library
  hydra16.kicad_sym with sym-lib-table.

PCB updated from the schematic. Includes pending changes to the counter,
bus breakout and memory daughter card projects.

Firmware:
- Remove S_REGISTER; T/U/V/W now at $FFF0-$FFF3 to match the hardware.
- Add math.s and sound.s (included by os_main.s).
- Rebuild the 65C02 ROM image.

Co-Authored-By: Claude Opus 5.5 <noreply@anthropic.com>
Parts:
- added H1, H3, H4: MountingHole, MountingHole:MountingHole_3.2mm_M3, symbol Mechanical:MountingHole
- added H2: MountingHole_Pad, MountingHole:MountingHole_3.2mm_M3_ISO7380_Pad_TopBottom, symbol Mechanical:MountingHole_Pad
Connections:
- net +5V: now also J17.79 (Pin_79)
- net GND: now also J17.78 (Pin_78), J18.77 (Pin_77), J18.78 (Pin_78), J19.77 (Pin_77), J19.78 (Pin_78), J20.77 (Pin_77), J20.78 (Pin_78), J21.77 (Pin_77), J21.78 (Pin_78), J22.77 (Pin_77), J22.78 (Pin_78), J23.77 (Pin_77), J23.78 (Pin_78), J24.77 (Pin_77), J24.78 (Pin_78), J25.77 (Pin_77), J25.78 (Pin_78), J26.77 (Pin_77), J26.78 (Pin_78), J27.77 (Pin_77), J27.78 (Pin_78), J28.77 (Pin_77), J28.78 (Pin_78), J29.77 (Pin_77), J29.78 (Pin_78), J30.77 (Pin_77), J30.78 (Pin_78), J31.77 (Pin_77), J31.78 (Pin_78), J32.77 (Pin_77), J32.78 (Pin_78), J33.77 (Pin_77), J33.78 (Pin_78), J34.77 (Pin_77), J34.78 (Pin_78), H2.1; no longer J17.79 (Pin_79)
Other:
- moved on the sheet: J32
