File: board/vera-x/vera-x.kicad_sch (KiCad schematic)
At the start: 25 parts, among them J1 VERA X 6.1 (2x13 socket), J10 Breakout J10: I2C, J11 Breakout J11: power (pin 3 is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, J12 PS/2 keyboard, J13 PS/2 mouse, J2 Breakout J2: data bus, J3 Breakout J3: address bus (A15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, J5 Breakout J5: interrupts & I/O, J6 Breakout J6: clocks, J7 Breakout J7: bus control (pin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, J8 Breakout J8: reset, J9 Breakout J9: audio, SW1 Power (press once at power-up), U1 74AHCT138, U2 74ACT00, U3 74AHCT245, U4 ATtiny861 (x16-smc)

Commit message: V1.8D board enhancements (1.8C software compatible)
Other:
- note added: "Never use breakout J11 pin 3: slot 0 carries -5 V there (the card labels it +5VA). Breakout J7 pin 5 is /DMAB (slot pin 23), not an inverted R/W: the strobes use RWB (J7 pin 4). Keep the bus wires short (15 cm or less); a ground wire beside PHI2. Plug and unplug with the power off. The wiring guide: docs/02-hardware/cards.md, the glue board (timing, bring-up, the SMC's firmware)."
- note removed: "Never use breakout J11 pin 3: slot 0 carries -5 V there (the card labels it +5VA). Breakout J7 pin 5 is /DMAB (slot pin 23), not an inverted R/W: the strobes use RWB (J7 pin 4). Keep the bus wires short (15 cm or less); a ground wire beside PHI2. Plug and unplug with the power off. The wiring guide: reborn/docs/vera-wiring.md (timing, bring-up, the SMC's firmware)."
Changed lines of the file:
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@@
 		(rev "1")
 		(company "Hydra-16")
-		(comment 1 "From reborn/docs/vera-wiring.md (slot 0; U3 optional, DNP)")
+		(comment 1 "From docs/02-hardware/cards.md (slot 0; U3 optional, DNP)")
 	)
 	(symbol
@@
 		)
 	)
-	(text "Never use breakout J11 pin 3: slot 0 carries -5 V there (the card labels it +5VA).\nBreakout J7 pin 5 is /DMAB (slot pin 23), not an inverted R/W: the strobes use RWB (J7 pin 4).\nKeep the bus wires short (15 cm or less); a ground wire beside PHI2. Plug and unplug with the power off.\nThe wiring guide: reborn/docs/vera-wiring.md (timing, bring-up, the SMC's firmware)."
+	(text "Never use breakout J11 pin 3: slot 0 carries -5 V there (the card labels it +5VA).\nBreakout J7 pin 5 is /DMAB (slot pin 23), not an inverted R/W: the strobes use RWB (J7 pin 4).\nKeep the bus wires short (15 cm or less); a ground wire beside PHI2. Plug and unplug with the power off.\nThe wiring guide: docs/02-hardware/cards.md, the glue board (timing, bring-up, the SMC's firmware)."
 		(exclude_from_sim no)
 		(at 302.26 203.2 0)
